File: Design Files/ap_io.kicad_sch (KiCad schematic)
At the start: 11 parts, among them J16 Conn_01x06_MountingPin, J17 Conn_01x06_MountingPin, J18 Conn_01x06_MountingPin, J19 Conn_01x06_MountingPin, U18 PCA9685PW

Commit message: New approach
Parts:
- removed C36, C37: 100nF, Capacitor_SMD:C_0402_1005Metric, symbol Device:C_Small_US
- removed J16, J17, J18, J19: Conn_01x06_MountingPin, Connector_JST:JST_GH_SM06B-GHS-TB_1x06-1MP_P1.25mm_Horizontal, symbol Connector_Generic_MountingPin:Conn_01x06_MountingPin
- removed RN1, RN2, RN3, RN4: R_Pack04, Package_SO:MSOP-8_3x3mm_P0.65mm, symbol Device:R_Pack04
- removed U18: PCA9685PW, Package_SO:TSSOP-28_4.4x9.7mm_P0.65mm, symbol Driver_LED:PCA9685PW
Connections:
- no-connect marks 4 -> 0
Other:
- note removed: "3.3V IO"
