File: Design Files/sensors.kicad_sch (KiCad schematic)
At the start: 22 parts, among them U10 BMI270, U11 74LVC2T45DC, U12 74LVC2T45DC, U15 AK09918C, U16 74LVC2T45DC, U20 MMC5983MA, U24 TCA9517ADGK, U25 BMP390

Commit message: New approach
Parts:
- removed C34, C35, C55, C57, C58, C59, C60, C61, C62: 100nF, Capacitor_SMD:C_0402_1005Metric, symbol Device:C_Small_US
- removed C63: 10uF, Capacitor_SMD:C_0402_1005Metric, symbol Device:C_Small_US
- removed R15, R16, R17, R22: 10k, Resistor_SMD:R_0402_1005Metric_Pad0.72x0.64mm_HandSolder, symbol Device:R_US
- removed U10: BMI270, SiGe_Lib:BMI270_BOS, symbol SiGe_Lib:BMI270
- removed U11, U12, U16: 74LVC2T45DC, Package_SO:VSSOP-8_2.3x2mm_P0.5mm, symbol Logic_LevelTranslator:74LVC2T45DC
- removed U15: AK09918C, SiGe_Lib:BGA4_WL-CSP_AKM, symbol SiGe_Lib:AK09918C
- removed U20: MMC5983MA, SiGe_Lib:MMC5983MA_MEM, symbol SiGe_Lib:MMC5983MA
- removed U24: TCA9517ADGK, Package_SO:VSSOP-8_3x3mm_P0.65mm, symbol Logic_LevelTranslator:TCA9517ADGK
- removed U25: BMP390, SiGe_Lib:10LGA_2X2X0p75_BOS, symbol SiGe_Lib:BMP390
Connections:
- no-connect marks 10 -> 0
Other:
- note removed: "1.8V @ 2mA"
- note removed: "1.8V/3.3 @ 2mA"
- note removed: "3.3V @ 2mA"
- note removed: "Internally Pulled to VCCB"
- note removed: "L = B to A H = A to B TODO: Finish setting up. Need dual 1bit for remainder of bus"
