File: Design Files/CM5_GPIO.kicad_sch (KiCad schematic)
At the start: 14 parts, among them J14 Micro_SD_Card_Det, J5 Conn_01x04_MountingPin, U1 RT9742GGJ5

Commit message: New approach
Parts:
- J14: footprint CM5IO:SDCARD_MOLEX_503398-1892 -> Connector_Card:microSD_HC_Molex_104031-0811
Changed lines of the file:
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@@
 			)
 		)
-		(property "Footprint" "CM5IO:SDCARD_MOLEX_503398-1892"
+		(property "Footprint" "Connector_Card:microSD_HC_Molex_104031-0811"
 			(at 356.87 110.49 0)
 			(hide yes)

Commit message: Checkin
Connections:
- net TRD1_N: now also TR1.14 (TD+); no longer TR1.16 (TD-)
- net TRD1_P: now also TR1.16 (TD-); no longer TR1.14 (TD+)
- net TRD1_RX_N: now also TR1.3 (TX+); no longer TR1.1 (TX-)
- net TRD1_RX_P: now also TR1.1 (TX-); no longer TR1.3 (TX+)
Changed lines of the file:
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@@
 	(wire
 		(pts
-			(xy 298.45 58.42) (xy 269.24 58.42)
-		)
-		(stroke
-			(width 0)
-			(type default)
-		)
-	)
-	(wire
-		(pts
 			(xy 78.74 133.35) (xy 88.9 133.35)
 		)
@@
 		)
 	)
+	(wire
+		(pts
+			(xy 298.45 53.34) (xy 298.45 50.8)
+		)
+		(stroke
+			(width 0)
+			(type default)
+		)
+	)
 	(polyline
 		(pts
@@
 	(wire
 		(pts
+			(xy 269.24 58.42) (xy 294.64 58.42)
+		)
+		(stroke
+			(width 0)
+			(type default)
+		)
+	)
+	(wire
+		(pts
 			(xy 149.86 54.61) (xy 163.83 54.61)
 		)
@@
 	(wire
 		(pts
+			(xy 294.64 58.42) (xy 294.64 45.72)
+		)
+		(stroke
+			(width 0)
+			(type default)
+		)
+	)
+	(wire
+		(pts
 			(xy 149.86 123.19) (xy 149.86 125.73)
 		)
@@
 	(wire
 		(pts
-			(xy 298.45 50.8) (xy 298.45 58.42)
-		)
-		(stroke
-			(width 0)
-			(type default)
-		)
-	)
-	(wire
-		(pts
 			(xy 269.24 45.72) (xy 285.75 45.72)
 		)
@@
 	(wire
 		(pts
-			(xy 294.64 45.72) (xy 294.64 53.34)
-		)
-		(stroke
-			(width 0)
-			(type default)
-		)
-	)
-	(wire
-		(pts
-			(xy 294.64 53.34) (xy 269.24 53.34)
+			(xy 269.24 53.34) (xy 298.45 53.34)
 		)
 		(stroke
@@
 		)
 	)
-	(label "TRD1_P"
+	(label "TRD1_N"
 		(at 238.76 53.34 0)
 		(effects
@@
 		)
 	)
-	(label "TRD1_N"
+	(label "TRD1_P"
 		(at 238.76 58.42 0)
 		(effects
@@
 		)
 	)
-	(label "TRD1_RX_P"
+	(label "TRD1_RX_N"
 		(at 271.78 53.34 0)
 		(effects
@@
 		)
 	)
-	(label "TRD1_RX_N"
-		(at 287.02 58.42 0)
+	(label "TRD1_RX_P"
+		(at 278.13 58.42 0)
 		(effects
 			(font
