File: Design Files/CM5_GPIO.kicad_sch (KiCad schematic)
At the start: 14 parts, among them J14 Micro_SD_Card_Det, J5 Conn_01x04_MountingPin, U1 RT9742GGJ5

Commit message: major fixes
Connections:
- net GND: no longer Module1.93 (nRPIBOOT)
- net SPI_CIPO0: now also Module1.40 (GPIO9); no longer Module1.44 (GPIO10)
- net SPI_CIPO1: now also Module1.26 (GPIO19); no longer Module1.27 (GPIO20)
- net SPI_COPI0: now also Module1.44 (GPIO10); no longer Module1.40 (GPIO9)
- net SPI_COPI1: now also Module1.27 (GPIO20); no longer Module1.26 (GPIO19)
- net GPIO25 renamed CAN_nINT
- new net nRPIBOOT: Module1.93 (nRPIBOOT)
Other:
- note removed: "Force RPIBOOT = Jumper Pins 1-2"
Changed lines of the file:
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@@
 		)
 	)
-	(text "Force RPIBOOT = Jumper Pins 1-2 \n"
-		(exclude_from_sim no)
-		(at 106.045 165.1 0)
-		(effects
-			(font
-				(size 1.27 1.27)
-			)
-			(justify right bottom)
-		)
-	)
 	(text "PWR LED"
 		(exclude_from_sim no)
@@
 	(wire
 		(pts
-			(xy 67.31 175.26) (xy 77.47 175.26)
-		)
-		(stroke
-			(width 0)
-			(type solid)
-		)
-	)
-	(wire
-		(pts
 			(xy 149.86 120.65) (xy 163.83 120.65)
 		)
@@
 	(wire
 		(pts
-			(xy 90.17 175.26) (xy 104.14 175.26)
-		)
-		(stroke
-			(width 0)
-			(type solid)
-		)
-	)
-	(wire
-		(pts
 			(xy 73.66 95.25) (xy 88.9 95.25)
 		)
@@
 	(wire
 		(pts
-			(xy 67.31 172.72) (xy 104.14 172.72)
-		)
-		(stroke
-			(width 0)
-			(type solid)
-		)
-	)
-	(wire
-		(pts
 			(xy 297.18 153.67) (xy 295.91 153.67)
 		)
@@
 	(wire
 		(pts
-			(xy 67.31 172.72) (xy 67.31 175.26)
-		)
-		(stroke
-			(width 0)
-			(type default)
-		)
-	)
-	(wire
-		(pts
 			(xy 260.35 130.81) (xy 260.35 132.08)
 		)
@@
 		)
 	)
-	(label "GPIO25"
-		(at 160.02 74.93 180)
-		(effects
-			(font
-				(size 1.27 1.27)
-			)
-			(justify right bottom)
-		)
-	)
 	(label "SD_DAT0"
 		(at 161.29 102.87 180)
@@
 		)
 	)
-	(label "GND"
-		(at 72.39 172.72 180)
-		(effects
-			(font
-				(size 1.27 1.27)
-			)
-			(justify right bottom)
-		)
-	)
 	(label "TRD1_P"
 		(at 238.76 58.42 0)
@@
 		)
 	)
-	(label "nRPIBOOT"
-		(at 100.076 172.72 180)
-		(effects
-			(font
-				(size 1.27 1.27)
-			)
-			(justify right bottom)
-		)
-	)
 	(label "3V3"
 		(at 198.12 93.98 180)
@@
 		)
 	)
-	(label "EEPROM_nWP"
-		(at 103.378 175.26 180)
-		(effects
-			(font
-				(size 1.27 1.27)
-			)
-			(justify right bottom)
-		)
-	)
 	(label "TRD0_TX_P"
 		(at 271.78 43.18 0)
@@
 		)
 	)
-	(label "GND"
-		(at 72.39 175.26 180)
-		(effects
-			(font
-				(size 1.27 1.27)
-			)
-			(justify right bottom)
-		)
-	)
 	(label "SD_CLK"
 		(at 273.05 128.27 0)
@@
 		)
 	)
-	(hierarchical_label "SPI_CIPO1"
+	(hierarchical_label "SPI_COPI1"
 		(shape input)
 		(at 163.83 57.15 0)
@@
 		)
 	)
+	(hierarchical_label "CAN_nINT"
+		(shape input)
+		(at 163.83 74.93 0)
+		(effects
+			(font
+				(size 1.27 1.27)
+			)
+			(justify left)
+		)
+	)
 	(hierarchical_label "SPI_0_CE0"
 		(shape output)
@@
 		)
 	)
-	(hierarchical_label "SPI_COPI0"
+	(hierarchical_label "SPI_CIPO0"
 		(shape output)
 		(at 73.66 72.39 180)
@@
 		)
 	)
-	(hierarchical_label "SPI_CIPO0"
+	(hierarchical_label "SPI_COPI0"
 		(shape input)
 		(at 73.66 77.47 180)
@@
 		)
 	)
-	(hierarchical_label "SPI_COPI1"
+	(hierarchical_label "SPI_CIPO1"
 		(shape output)
 		(at 73.66 54.61 180)

Commit message: Ehh, mostly there...
Parts:
- removed NT1: NetTie_2, NetTie:NetTie-2_SMD_Pad0.5mm, symbol Device:NetTie_2
- added C36: 100nF, Capacitor_SMD:C_0603_1608Metric_Pad1.08x0.95mm_HandSolder, symbol Device:C_Small_US
- added R22, R28, R29, R30, R31, R32: 4.7k, Resistor_SMD:R_0402_1005Metric_Pad0.72x0.64mm_HandSolder, symbol Device:R_US
- added U10: AT24C256C-SSHL-T, SiGe_Lib:8S1_MCH, symbol Memory_EEPROM:AT24CS64-MAHM
- C3, C54, C56, D4, R19, R20, R21, R4: KiLib_Generator (none) -> SMD_2terminal_chip_molded
- J5: KiLib_Generator (none) -> connector/SMD_single_row_plus_mounting_pad
- TR1, U1: KiLib_Generator (none) -> package/gullwing
Connections:
- net GPIO_VREF is gone; now on net 3V3_Peripheral: Module1.78 (GPIO_VREF(1.8v/3.3v_Input))
- net 3V3_Peripheral: now also C36.1, R22.1, R28.1, R29.1, R30.1, R31.1, R32.1, U10.8 (VCC)
- net GND: now also C36.2, U10.1 (A0), U10.2 (A1), U10.3 (A2), U10.4 (GND), U10.9 (GND)
- net ID_SC: now also R31.2, U10.6 (SCL)
- net ID_SD: now also R30.2, U10.5 (SDA)
- net SCL4: now also R29.2
- net SDA4: now also R28.2
- net PMIC_nINT: now reaches Module1.24 (GPIO26)
- net PMIC_nINT: now also R22.2
- new net: R32.2, U10.7 (WP)
