File: Design Files/compactPi.kicad_sch (KiCad schematic)
At the start: 7 parts, among them J15 USB_C_Receptacle_USB2.0, U22 WE-TVS-82400102

Commit message: some stuff fixed
Connections:
- no-connect marks 17 -> 15
Changed lines of the file:
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@@
-	)
-	(no_connect
-		(at 49.53 140.97)
-	)
-	(no_connect
-		(at 49.53 138.43)
 	)
 	(no_connect
@@
 	(wire
 		(pts
+			(xy 39.37 138.43) (xy 49.53 138.43)
+		)
+		(stroke
+			(width 0)
+			(type default)
+		)
+	)
+	(wire
+		(pts
 			(xy 146.05 90.17) (xy 163.83 90.17)
 		)
@@
 		(pts
 			(xy 308.61 138.43) (xy 322.58 138.43)
+		)
+		(stroke
+			(width 0)
+			(type default)
+		)
+	)
+	(wire
+		(pts
+			(xy 39.37 140.97) (xy 49.53 140.97)
 		)
 		(stroke
@@
 		)
 	)
-	(label "5V_PERIPHERAL"
+	(label "5V0_PERIPHERAL"
 		(at 114.3 128.27 180)
 		(effects
@@
 		)
 	)
+	(label "CC1"
+		(at 39.37 140.97 0)
+		(effects
+			(font
+				(size 1.27 1.27)
+			)
+			(justify left bottom)
+		)
+	)
 	(label "USB2_P"
 		(at 86.36 63.5 180)
@@
 		(effects
 			(font
+				(size 1.27 1.27)
+			)
+			(justify left bottom)
+		)
+	)
+	(label "CC2"
+		(at 39.37 138.43 0)
+		(effects
+			(font

Commit message: major fixes
Parts:
- R12: value 2.2K 1% -> 10k
Other:
- sheet CM5 GPIO Ethernet SDIO ports: added CAN_nINT; removed none
- sheet CM5 USB HDMI ports: added 5V0_PERIPHERAL; removed 5V0_Peripheral
- sheet Power ports: added 3V3_IN; removed none
Changed lines of the file:
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@@
+	(wire
+		(pts
+			(xy 39.37 128.27) (xy 49.53 128.27)
+		)
+		(stroke
+			(width 0)
+			(type default)
+		)
+	)
 	(wire
 		(pts
@@
 	(wire
 		(pts
+			(xy 220.98 151.13) (xy 234.95 151.13)
+		)
+		(stroke
+			(width 0)
+			(type default)
+		)
+	)
+	(wire
+		(pts
 			(xy 220.98 156.21) (xy 234.95 156.21)
 		)
@@
 		(pts
 			(xy 148.59 143.51) (xy 163.83 143.51)
+		)
+		(stroke
+			(width 0)
+			(type default)
+		)
+	)
+	(wire
+		(pts
+			(xy 308.61 148.59) (xy 322.58 148.59)
 		)
 		(stroke
@@
 		)
 	)
+	(label "CAN_nINT"
+		(at 308.61 148.59 0)
+		(effects
+			(font
+				(size 1.27 1.27)
+			)
+			(justify left bottom)
+		)
+	)
 	(label "5V0_CORE"
 		(at 234.95 143.51 180)
@@
 		)
 	)
+	(label "CAN_nINT"
+		(at 234.95 151.13 180)
+		(effects
+			(font
+				(size 1.27 1.27)
+			)
+			(justify right bottom)
+		)
+	)
 	(label "I2C_INT_SDA0"
 		(at 148.59 130.81 0)
@@
 		)
 	)
-	(label "5V_Peripheral"
+	(label "5V0_PERIPHERAL"
 		(at 146.05 90.17 0)
+		(effects
+			(font
+				(size 1.27 1.27)
+			)
+			(justify left bottom)
+		)
+	)
+	(label "3V3"
+		(at 39.37 128.27 0)
 		(effects
 			(font
@@
 		(dnp no)
 		(property "Reference" "R12"
-			(at 72.898 47.625 0)
-			(show_name no)
-			(do_not_autoplace no)
-			(effects
-				(font
-					(size 1.27 1.27)
-				)
-				(justify left)
-			)
-		)
-		(property "Value" "2.2K 1%"
-			(at 67.818 49.53 0)
+			(at 71.882 47.498 0)
+			(show_name no)
+			(do_not_autoplace no)
+			(effects
+				(font
+					(size 1.27 1.27)
+				)
+				(justify left)
+			)
+		)
+		(property "Value" "10k"
+			(at 71.882 49.022 0)
 			(show_name no)
 			(do_not_autoplace no)
@@
 			)
 		)
+		(pin "CAN_nINT" input
+			(at 220.98 151.13 0)
+			(effects
+				(font
+					(size 1.27 1.27)
+				)
+				(justify right)
+			)
+		)
 		(instances
 			(project "compactPi"
@@
 			)
 		)
-		(pin "5V0_Peripheral" input
+		(pin "5V0_PERIPHERAL" input
 			(at 163.83 90.17 180)
 			(effects
@@
 			)
 		)
+		(pin "3V3_IN" input
+			(at 49.53 128.27 180)
+			(effects
+				(font
+					(size 1.27 1.27)
+				)
+				(justify left)
+			)
+		)

Commit message: Ehh, mostly there...
Parts:
- H1, H2, H3, H4: KiLib_Generator (none) -> mounting_hardware/mounting_hole
- R12: KiLib_Generator (none) -> SMD_2terminal_chip_molded
- U22: KiLib_Generator (none) -> package/gullwing
Other:
- sheet CM5 GPIO Ethernet SDIO ports: added PMIC_nINT; removed GPIO_VREF, ID_SC, ID_SD
- sheet CM5 USB HDMI ports: added 3V3; removed GPIO_VREF, ID_SC, ID_SD
- sheet Power ports: added I2C_PMIC_SCL, I2C_PMIC_SDA, I2C_PMIC_nINT; removed 5V_PERIPHERAL
Changed lines of the file:
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@@
-	(wire
-		(pts
-			(xy 214.63 111.76) (xy 214.63 127)
-		)
-		(stroke
-			(width 0)
-			(type solid)
-		)
-	)
 	(wire
 		(pts
@@
 	(wire
 		(pts
+			(xy 146.05 97.79) (xy 163.83 97.79)
+		)
+		(stroke
+			(width 0)
+			(type default)
+		)
+	)
+	(wire
+		(pts
 			(xy 151.13 156.21) (xy 163.83 156.21)
 		)
@@
 	(wire
 		(pts
-			(xy 184.15 111.76) (xy 184.15 127)
-		)
-		(stroke
-			(width 0)
-			(type solid)
-		)
-	)
-	(wire
-		(pts
 			(xy 220.98 148.59) (xy 234.95 148.59)
 		)
@@
 	(wire
 		(pts
+			(xy 34.29 147.32) (xy 49.53 147.32)
+		)
+		(stroke
+			(width 0)
+			(type default)
+		)
+	)
+	(wire
+		(pts
 			(xy 52.07 45.72) (xy 77.47 45.72)
 		)
@@
 	(wire
 		(pts
-			(xy 180.34 111.76) (xy 180.34 127)
-		)
-		(stroke
-			(width 0)
-			(type solid)
-		)
-	)
-	(wire
-		(pts
 			(xy 220.98 143.51) (xy 234.95 143.51)
 		)
@@
 	(wire
 		(pts
+			(xy 34.29 152.4) (xy 49.53 152.4)
+		)
+		(stroke
+			(width 0)
+			(type default)
+		)
+	)
+	(wire
+		(pts
 			(xy 308.61 140.97) (xy 322.58 140.97)
 		)
@@
 	(wire
 		(pts
+			(xy 34.29 149.86) (xy 49.53 149.86)
+		)
+		(stroke
+			(width 0)
+			(type default)
+		)
+	)
+	(wire
+		(pts
 			(xy 308.61 130.81) (xy 322.58 130.81)
 		)
@@
 	(wire
 		(pts
+			(xy 148.59 148.59) (xy 163.83 148.59)
+		)
+		(stroke
+			(width 0)
+			(type default)
+		)
+	)
+	(wire
+		(pts
 			(xy 308.61 146.05) (xy 322.58 146.05)
 		)
@@
 			(width 0)
 			(type default)
+		)
+	)
+	(label "I2C_PMIC_SDA"
+		(at 34.29 149.86 0)
+		(effects
+			(font
+				(size 1.27 1.27)
+			)
+			(justify left bottom)
+		)
+	)
+	(label "I2C_PMIC_nINT"
+		(at 34.29 152.4 0)
+		(effects
+			(font
+				(size 1.27 1.27)
+			)
+			(justify left bottom)
 		)
 	)
@@
 		)
 	)
+	(label "3V3"
+		(at 146.05 97.79 0)
+		(effects
+			(font
+				(size 1.27 1.27)
+			)
+			(justify left bottom)
+		)
+	)
 	(label "USB2a_N"
 		(at 153.67 66.04 0)
@@
 		)
 	)
+	(label "I2C_PMIC_SCL"
+		(at 34.29 147.32 0)
+		(effects
+			(font
+				(size 1.27 1.27)
+			)
+			(justify left bottom)
+		)
+	)
 	(label "CAN_nINT"
 		(at 234.95 151.13 180)
@@
 		)
 	)
-	(label "I2C_PWM_SCL"
+	(label "I2C_PMIC_SCL"
 		(at 148.59 146.05 0)
 		(effects
@@
 		)
 	)
-	(label "I2C_PWM_SDA"
+	(label "I2C_PMIC_nINT"
+		(at 148.59 148.59 0)
+		(effects
+			(font
+				(size 1.27 1.27)
+			)
+			(justify left bottom)
+		)
+	)
+	(label "I2C_PMIC_SDA"
 		(at 148.59 143.51 0)
 		(effects
@@
 			)
 		)
+		(property "KiLib_Generator" "mounting_hardware/mounting_hole"
+			(at 38.1 276.86 0)
+			(hide yes)
+			(show_name no)
+			(do_not_autoplace no)
+			(effects
+				(font
+					(size 1.27 1.27)
+				)
+			)
+		)
 		(pin "1"
 		)
@@
 			)
 		)
+		(property "KiLib_Generator" "mounting_hardware/mounting_hole"
+			(at 38.1 264.16 0)
+			(hide yes)
+			(show_name no)
+			(do_not_autoplace no)
+			(effects
+				(font
+					(size 1.27 1.27)
+				)
+			)
+		)
 		(pin "1"
 		)
@@
 			)
 		)
+		(property "KiLib_Generator" "package/gullwing"
+			(at 93.98 60.96 0)
+			(hide yes)
+			(show_name no)
+			(do_not_autoplace no)
+			(effects
+				(font
+					(size 1.27 1.27)
+				)
+			)
+		)
 		(pin "3"
 		)
@@
 			)
 		)
+		(property "KiLib_Generator" "mounting_hardware/mounting_hole"
+			(at 59.69 264.16 0)
+			(hide yes)
+			(show_name no)
+			(do_not_autoplace no)
+			(effects
+				(font
+					(size 1.27 1.27)
+				)
+			)
+		)
 		(pin "1"
 		)
@@
 		)
 		(property "Field8" ""
+			(at 77.47 49.53 0)
+			(hide yes)
+			(show_name no)
+			(do_not_autoplace no)
+			(effects
+				(font
+					(size 1.27 1.27)
+				)
+			)
+		)
+		(property "KiLib_Generator" "SMD_2terminal_chip_molded"
 			(at 77.47 49.53 0)
 			(hide yes)
@@
 			)
 		)
+		(property "KiLib_Generator" "mounting_hardware/mounting_hole"
+			(at 59.69 276.86 0)
+			(hide yes)
+			(show_name no)
+			(do_not_autoplace no)
+			(effects
+				(font
+					(size 1.27 1.27)
+				)
+			)
+		)
 		(pin "1"
 		)
@@
 			)
 		)
-		(pin "ID_SC" output
-			(at 184.15 127 90)
-			(effects
-				(font
-					(size 1.27 1.27)
-				)
-				(justify right)
-			)
-		)
-		(pin "ID_SD" output
-			(at 180.34 127 90)
-			(effects
-				(font
-					(size 1.27 1.27)
-				)
-				(justify right)
-			)
-		)
 		(pin "SCL0" output
 			(at 163.83 133.35 180)
@@
 			)
 		)
-		(pin "GPIO_VREF" output
-			(at 214.63 127 90)
-			(effects
-				(font
-					(size 1.27 1.27)
-				)
-				(justify right)
-			)
-		)
 		(pin "SPI_CIPO0" input
 			(at 163.83 161.29 180)
@@
 				)
 				(justify right)
+			)
+		)
+		(pin "PMIC_nINT" input
+			(at 163.83 148.59 180)
+			(effects
+				(font
+					(size 1.27 1.27)
+				)
+				(justify left)
 			)
 		)
@@
 			)
 		)
-		(pin "ID_SC" input
-			(at 184.15 111.76 270)
-			(effects
-				(font
-					(size 1.27 1.27)
-				)
-				(justify left)
-			)
-		)
-		(pin "ID_SD" input
-			(at 180.34 111.76 270)
-			(effects
-				(font
-					(size 1.27 1.27)
-				)
-				(justify left)
-			)
-		)
 		(pin "PCIE_CLK_P" output
 			(at 220.98 72.39 0)
@@
 			)
 		)
-		(pin "GPIO_VREF" input
-			(at 214.63 111.76 270)
-			(effects
-				(font
-					(size 1.27 1.27)
-				)
-				(justify left)
-			)
-		)
 		(pin "PCIE_PWR_EN" output
 			(at 220.98 87.63 0)
@@
 		(pin "5V0_PERIPHERAL" input
 			(at 163.83 90.17 180)
+			(effects
+				(font
+					(size 1.27 1.27)
+				)
+				(justify left)
+			)
+		)
+		(pin "3V3" input
+			(at 163.83 97.79 180)
 			(effects
 				(font
@@
 	(sheet
 		(at 49.53 120.65)
-		(size 40.64 22.86)
+		(size 40.64 39.37)
 		(exclude_from_sim no)
 		(in_bom yes)
@@
 		)
 		(property "Sheetfile" "Power.kicad_sch"
-			(at 49.53 144.0946 0)
+			(at 49.53 160.6046 0)
 			(show_name no)
 			(do_not_autoplace no)
@@
 			)
 		)
-		(pin "5V_PERIPHERAL" bidirectional
-			(at 90.17 139.7 0)
-			(effects
-				(font
-					(size 1.27 1.27)
-				)
-				(justify right)
-			)
-		)
 		(pin "3V3_IN" input
 			(at 49.53 128.27 180)
 			(effects
 				(font
+					(size 1.27 1.27)
+				)
+				(justify left)
+			)
+		)
+		(pin "I2C_PMIC_SCL" bidirectional
+			(at 49.53 147.32 180)
+			(effects
+				(font
+					(size 1.27 1.27)
+				)
+				(justify left)
+			)
+		)
+		(pin "I2C_PMIC_nINT" output
+			(at 49.53 152.4 180)
+			(effects
+				(font
+					(size 1.27 1.27)
+				)
+				(justify left)
+			)
+		)
+		(pin "I2C_PMIC_SDA" bidirectional
+			(at 49.53 149.86 180)
+			(effects
+				(font
