File: Design Files/autopilot_conn.kicad_sch (KiCad schematic)
At the start: 26 parts, among them J10 Conn_01x06_MountingPin, J12 Conn_01x02_MountingPin, J13 Conn_01x02_MountingPin, J3 Conn_01x04_MountingPin, J4 Conn_01x06_MountingPin, J6 Conn_01x04_MountingPin, J7 Conn_01x04_MountingPin, J8 Conn_01x04_MountingPin, J9 Conn_01x04_MountingPin, U21 MCP25625x-x-ML, Y1 Crystal_GND24_Small

Commit message: New approach
Parts:
- removed J12, J13: Conn_01x02_MountingPin, Connector_JST:JST_GH_BM02B-GHS-TBT_1x02-1MP_P1.25mm_Vertical, symbol Connector_Generic_MountingPin:Conn_01x02_MountingPin
- removed J3: Conn_01x04_MountingPin, Connector_JST:JST_GH_BM04B-GHS-TBT_1x04-1MP_P1.25mm_Vertical, symbol Connector_Generic_MountingPin:Conn_01x04_MountingPin
Connections:
- no-connect marks 13 -> 10
Other:
- note removed: "ADC"
- note removed: "LEAK"

Commit message: some stuff fixed
Parts:
- added R27: 10k, Resistor_SMD:R_0402_1005Metric_Pad0.72x0.64mm_HandSolder, symbol Device:R_US
Connections:
- net 3V3: now also R27.1
- net CAN_RST: now also R27.2
Other:
- moved on the sheet: R23
Changed lines of the file:
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@@
 	)
 	(junction
+		(at 194.31 100.33)
+		(diameter 0)
+		(color 0 0 0 0)
+	)
+	(junction
 		(at 220.98 33.02)
 		(diameter 0)
@@
 	)
 	(junction
-		(at 232.41 100.33)
+		(at 196.85 100.33)
 		(diameter 0)
 		(color 0 0 0 0)
@@
 	(wire
 		(pts
-			(xy 223.52 100.33) (xy 232.41 100.33)
+			(xy 187.96 100.33) (xy 194.31 100.33)
 		)
 		(stroke
@@
 	(wire
 		(pts
+			(xy 196.85 100.33) (xy 240.03 100.33)
+		)
+		(stroke
+			(width 0)
+			(type default)
+		)
+	)
+	(wire
+		(pts
 			(xy 53.34 30.48) (xy 66.04 30.48)
 		)
@@
 	(wire
 		(pts
-			(xy 58.42 152.4) (xy 58.42 146.05)
+			(xy 189.23 87.63) (xy 194.31 87.63)
 		)
 		(stroke
@@
 	(wire
 		(pts
-			(xy 234.95 85.09) (xy 240.03 85.09)
+			(xy 58.42 152.4) (xy 58.42 146.05)
 		)
 		(stroke
@@
 	(wire
 		(pts
-			(xy 257.81 46.99) (xy 257.81 33.02)
+			(xy 234.95 85.09) (xy 240.03 85.09)
 		)
 		(stroke
@@
 	(wire
 		(pts
-			(xy 48.26 30.48) (xy 53.34 30.48)
+			(xy 257.81 46.99) (xy 257.81 33.02)
 		)
 		(stroke
@@
 	(wire
 		(pts
-			(xy 53.34 48.26) (xy 53.34 30.48)
+			(xy 48.26 30.48) (xy 53.34 30.48)
 		)
 		(stroke
@@
 	(wire
 		(pts
-			(xy 308.61 62.23) (xy 308.61 67.31)
+			(xy 53.34 48.26) (xy 53.34 30.48)
 		)
 		(stroke
@@
 	(wire
 		(pts
-			(xy 308.61 49.53) (xy 304.8 49.53)
+			(xy 308.61 62.23) (xy 308.61 67.31)
 		)
 		(stroke
@@
 	(wire
 		(pts
-			(xy 240.03 100.33) (xy 232.41 100.33)
+			(xy 308.61 49.53) (xy 304.8 49.53)
 		)
 		(stroke
@@
 	(wire
 		(pts
+			(xy 194.31 87.63) (xy 194.31 91.44)
+		)
+		(stroke
+			(width 0)
+			(type default)
+		)
+	)
+	(wire
+		(pts
 			(xy 308.61 67.31) (xy 300.99 67.31)
 		)
@@
 	(wire
 		(pts
-			(xy 232.41 100.33) (xy 232.41 102.87)
+			(xy 196.85 100.33) (xy 196.85 102.87)
 		)
 		(stroke
@@
 	(wire
 		(pts
+			(xy 194.31 100.33) (xy 196.85 100.33)
+		)
+		(stroke
+			(width 0)
+			(type default)
+		)
+	)
+	(wire
+		(pts
 			(xy 270.51 85.09) (xy 284.48 85.09)
 		)
@@
 	(wire
 		(pts
+			(xy 194.31 99.06) (xy 194.31 100.33)
+		)
+		(stroke
+			(width 0)
+			(type default)
+		)
+	)
+	(wire
+		(pts
 			(xy 293.37 66.04) (xy 299.72 66.04)
 		)
@@
 		)
 	)
+	(label "3V3"
+		(at 189.23 87.63 0)
+		(effects
+			(font
+				(size 1.27 1.27)
+			)
+			(justify left bottom)
+		)
+	)
 	(label "SPI_CAN_SCK_3V3"
 		(at 219.71 62.23 0)
@@
 	(hierarchical_label "CAN_RST"
 		(shape input)
-		(at 223.52 100.33 180)
+		(at 187.96 100.33 180)
 		(effects
 			(font
@@
 	(symbol
 		(lib_id "power:GND")
-		(at 232.41 110.49 0)
+		(at 196.85 110.49 0)
 		(unit 1)
 		(body_style 1)
@@
 		(dnp no)
 		(property "Reference" "#PWR064"
-			(at 232.41 116.84 0)
+			(at 196.85 116.84 0)
 			(hide yes)
 			(show_name no)
@@
 		)
 		(property "Value" "GND"
-			(at 232.537 114.8842 0)
+			(at 196.977 114.8842 0)
 			(show_name no)
 			(do_not_autoplace no)
@@
 		)
 		(property "Footprint" ""
-			(at 232.41 110.49 0)
+			(at 196.85 110.49 0)
 			(hide yes)
 			(show_name no)
@@
 		)
 		(property "Datasheet" ""
-			(at 232.41 110.49 0)
+			(at 196.85 110.49 0)
 			(hide yes)
 			(show_name no)
@@
 		)
 		(property "Description" "Power symbol creates a global label with name \"GND\" , ground"
-			(at 232.41 110.49 0)
+			(at 196.85 110.49 0)
 			(hide yes)
 			(show_name no)
@@
 	)
 	(symbol
+		(lib_id "Device:R_US")
+		(at 194.31 95.25 0)
+		(unit 1)
+		(body_style 1)
+		(exclude_from_sim no)
+		(in_bom yes)
+		(on_board yes)
+		(in_pos_files yes)
+		(dnp no)
+		(fields_autoplaced yes)
+		(property "Reference" "R27"
+			(at 196.85 93.9799 0)
+			(show_name no)
+			(do_not_autoplace no)
+			(effects
+				(font
+					(size 1.27 1.27)
+				)
+				(justify left)
+			)
+		)
+		(property "Value" "10k"
+			(at 196.85 96.5199 0)
+			(show_name no)
+			(do_not_autoplace no)
+			(effects
+				(font
+					(size 1.27 1.27)
+				)
+				(justify left)
+			)
+		)
+		(property "Footprint" "Resistor_SMD:R_0402_1005Metric_Pad0.72x0.64mm_HandSolder"
+			(at 195.326 95.504 90)
+			(hide yes)
+			(show_name no)
+			(do_not_autoplace no)
+			(effects
+				(font
+					(size 1.27 1.27)
+				)
+			)
+		)
+		(property "Datasheet" ""
+			(at 194.31 95.25 0)
+			(hide yes)
+			(show_name no)
+			(do_not_autoplace no)
+			(effects
+				(font
+					(size 1.27 1.27)
+				)
+			)
+		)
+		(property "Description" "Resistor, US symbol"
+			(at 194.31 95.25 0)
+			(hide yes)
+			(show_name no)
+			(do_not_autoplace no)
+			(effects
+				(font
+					(size 1.27 1.27)
+				)
+			)
+		)
+		(pin "2"
+		)
+		(pin "1"
+		)
+		(instances
+			(project "compactPi"
+				(path "/e63e39d7-6ac0-4ffd-8aa3-1841a4541b55/efe27aed-b9d7-4250-8fde-aaa7412d6a69"
+					(reference "R27")
+					(unit 1)
+				)
+			)
+		)
+	)
+	(symbol
 		(lib_id "Device:C_Small_US")
 		(at 213.36 35.56 0)
@@
 	(symbol
 		(lib_id "Device:R_US")
-		(at 232.41 106.68 0)
+		(at 196.85 106.68 0)
 		(unit 1)
 		(body_style 1)
@@
 		(fields_autoplaced yes)
 		(property "Reference" "R23"
-			(at 234.95 105.4099 0)
+			(at 199.39 105.4099 0)
 			(show_name no)
 			(do_not_autoplace no)
@@
 		)
 		(property "Value" "10k"
-			(at 234.95 107.9499 0)
+			(at 199.39 107.9499 0)
 			(show_name no)
 			(do_not_autoplace no)
@@
 		)
 		(property "Footprint" "Resistor_SMD:R_0402_1005Metric_Pad0.72x0.64mm_HandSolder"
-			(at 233.426 106.934 90)
+			(at 197.866 106.934 90)
 			(hide yes)
 			(show_name no)
@@
 		)
 		(property "Datasheet" ""
-			(at 232.41 106.68 0)
+			(at 196.85 106.68 0)
 			(hide yes)
 			(show_name no)
@@
 		)
 		(property "Description" "Resistor, US symbol"
-			(at 232.41 106.68 0)
+			(at 196.85 106.68 0)
 			(hide yes)
 			(show_name no)

Commit message: major fixes
Parts:
- added C69: 10u, Capacitor_SMD:C_0201_0603Metric, symbol Device:C_Small_US
- R23: now not fitted
Connections:
- net 3V3: now also U21.3 (V_{DD}), C69.1
- net 5V0: no longer U21.3 (V_{DD})
- net GND: now also C69.2
- net UART1_RX_In: now also J4.3 (Pin_3); no longer J4.2 (Pin_2)
- net UART1_TX_Out: now also J4.2 (Pin_2); no longer J4.3 (Pin_3)
- net UART2_RX_In: now also J10.3 (Pin_3); no longer J10.2 (Pin_2)
- net UART2_TX_Out: now also J10.2 (Pin_2); no longer J10.3 (Pin_3)
