File: Design Files/autopilot_conn.kicad_sch (KiCad schematic)
At the start: 25 parts, among them J10 Conn_01x06_MountingPin, J4 Conn_01x06_MountingPin, J6 Conn_01x04_MountingPin, J7 Conn_01x04_MountingPin, J8 Conn_01x04_MountingPin, J9 Conn_01x04_MountingPin, U21 MCP25625x-x-ML, Y1 Crystal_GND24_Small

Commit message: Ehh, mostly there...
Parts:
- C38, C39, C52, C53, C64, C65, C66, C67, C68, C69, R23, R24, R25, R26, R27: KiLib_Generator (none) -> SMD_2terminal_chip_molded
- D5: KiLib_Generator (none) -> package/gullwing
- J10, J4, J6, J7, J8, J9: KiLib_Generator (none) -> connector/SMD_single_row_plus_mounting_pad
- U21: KiLib_Generator (none) -> package/no_lead
- Y1: KiLib_Generator (none) -> crystal_resonator_oscillator; private KLC_S4.1 -> (none)
Connections:
- net unconnected-(J9-MountPin-PadMP)_1: now reaches J9.MP (MountPin)
