File: Design Files/CM5_HighSpeed.kicad_sch (KiCad schematic)
At the start: 9 parts, among them J11 Conn_01x04_MountingPin, J2 HDMI_A_1.4, U17 RT9742SNGV, U23 WE-TVS-82400102

Commit message: major fixes
Parts:
- added R18: 10k, Resistor_SMD:R_0402_1005Metric_Pad0.72x0.64mm_HandSolder, symbol Device:R_US
Connections:
- net GND: now also R18.2
- net VBUS_EN: now also R18.1
- net USB3-1-Port_N: now reaches J11.2 (Pin_2), U23.6
- net USB3-1-Port_P: now reaches J11.3 (Pin_3), U23.4
- net 5V0_Peripheral renamed 5V0_PERIPHERAL
Other:
- moved on the sheet: J11
Changed lines of the file:
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@@
 	)
 	(junction
+		(at 152.4 97.79)
+		(diameter 0)
+		(color 0 0 0 0)
+	)
+	(junction
 		(at 280.67 179.07)
 		(diameter 0)
@@
 	)
 	(no_connect
-		(at 207.01 163.83)
+		(at 218.44 163.83)
 	)
 	(wire
 		(pts
-			(xy 194.31 157.48) (xy 189.23 157.48)
+			(xy 256.54 207.01) (xy 262.89 207.01)
+		)
+		(stroke
+			(width 0)
+			(type solid)
+		)
+	)
+	(wire
+		(pts
+			(xy 193.04 157.48) (xy 189.23 157.48)
 		)
 		(stroke
@@
 	(wire
 		(pts
-			(xy 127 97.79) (xy 148.59 97.79)
+			(xy 127 97.79) (xy 152.4 97.79)
 		)
 		(stroke
@@
 	(wire
 		(pts
-			(xy 194.31 156.21) (xy 194.31 157.48)
+			(xy 193.04 156.21) (xy 193.04 157.48)
 		)
 		(stroke
@@
 	(wire
 		(pts
-			(xy 207.01 144.78) (xy 198.12 144.78)
+			(xy 220.98 143.51) (xy 198.12 143.51)
 		)
 		(stroke
@@
 	(wire
 		(pts
-			(xy 193.04 153.67) (xy 201.93 153.67)
+			(xy 193.04 153.67) (xy 213.36 153.67)
 		)
 		(stroke
@@
 	(wire
 		(pts
+			(xy 152.4 97.79) (xy 152.4 101.6)
+		)
+		(stroke
+			(width 0)
+			(type default)
+		)
+	)
+	(wire
+		(pts
 			(xy 238.76 102.87) (xy 262.89 102.87)
 		)
@@
 	(wire
 		(pts
-			(xy 198.12 151.13) (xy 201.93 151.13)
+			(xy 198.12 151.13) (xy 213.36 151.13)
 		)
 		(stroke
@@
 	(wire
 		(pts
-			(xy 198.12 144.78) (xy 198.12 151.13)
+			(xy 198.12 143.51) (xy 198.12 151.13)
 		)
 		(stroke
@@
 	(wire
 		(pts
-			(xy 201.93 156.21) (xy 194.31 156.21)
+			(xy 213.36 156.21) (xy 193.04 156.21)
 		)
 		(stroke
@@
 	(wire
 		(pts
-			(xy 257.81 207.01) (xy 262.89 207.01)
-		)
-		(stroke
-			(width 0)
-			(type solid)
-		)
-	)
-	(wire
-		(pts
 			(xy 280.67 133.35) (xy 280.67 134.62)
 		)
@@
 	(wire
 		(pts
+			(xy 152.4 97.79) (xy 158.75 97.79)
+		)
+		(stroke
+			(width 0)
+			(type solid)
+		)
+	)
+	(wire
+		(pts
 			(xy 129.54 161.29) (xy 129.54 168.91)
 		)
@@
 	(wire
 		(pts
-			(xy 201.93 158.75) (xy 200.66 158.75)
+			(xy 213.36 158.75) (xy 200.66 158.75)
 		)
 		(stroke
@@
 		)
 	)
+	(label "USB3-1-Port_N"
+		(at 193.04 153.67 0)
+		(effects
+			(font
+				(size 1.27 1.27)
+			)
+			(justify left bottom)
+		)
+	)
 	(label "HDMI0_D1_N"
 		(at 238.76 92.71 0)
@@
 		)
 	)
+	(label "USB3-1-Port_P"
+		(at 193.04 156.21 0)
+		(effects
+			(font
+				(size 1.27 1.27)
+			)
+			(justify left bottom)
+		)
+	)
 	(label "GPIO_VREF"
 		(at 263.525 163.83 0)
@@
 	(hierarchical_label "VBUS_EN"
 		(shape output)
-		(at 148.59 97.79 0)
+		(at 158.75 97.79 0)
 		(effects
 			(font
@@
 		)
 	)
-	(hierarchical_label "PCIE_PWR_EN"
-		(shape output)
-		(at 59.69 90.17 180)
+	(hierarchical_label "5V0_PERIPHERAL"
+		(shape input)
+		(at 256.54 207.01 180)
 		(effects
 			(font
@@
 		)
 	)
-	(hierarchical_label "PCIE_CLK_P"
+	(hierarchical_label "PCIE_PWR_EN"
 		(shape output)
-		(at 59.69 95.25 180)
+		(at 59.69 90.17 180)
 		(effects
 			(font
@@
 		)
 	)
-	(hierarchical_label "PCIE_RX_N"
-		(shape input)
-		(at 59.69 105.41 180)
+	(hierarchical_label "PCIE_CLK_P"
+		(shape output)
+		(at 59.69 95.25 180)
 		(effects
 			(font
@@
 		)
 	)
-	(hierarchical_label "5V0_Peripheral"
+	(hierarchical_label "PCIE_RX_N"
 		(shape input)
-		(at 257.81 207.01 180)
+		(at 59.69 105.41 180)
 		(effects
 			(font
@@
 		)
 	)
-	(hierarchical_label "5V0_Peripheral"
+	(hierarchical_label "5V0_PERIPHERAL"
 		(shape input)
-		(at 207.01 144.78 0)
+		(at 220.98 143.51 0)
 		(effects
 			(font
@@
 	)
 	(symbol
+		(lib_id "Device:R_US")
+		(at 152.4 105.41 0)
+		(unit 1)
+		(body_style 1)
+		(exclude_from_sim no)
+		(in_bom yes)
+		(on_board yes)
+		(in_pos_files yes)
+		(dnp no)
+		(fields_autoplaced yes)
+		(property "Reference" "R18"
+			(at 154.94 104.1399 0)
+			(show_name no)
+			(do_not_autoplace no)
+			(effects
+				(font
+					(size 1.27 1.27)
+				)
+				(justify left)
+			)
+		)
+		(property "Value" "10k"
+			(at 154.94 106.6799 0)
+			(show_name no)
+			(do_not_autoplace no)
+			(effects
+				(font
+					(size 1.27 1.27)
+				)
+				(justify left)
+			)
+		)
+		(property "Footprint" "Resistor_SMD:R_0402_1005Metric_Pad0.72x0.64mm_HandSolder"
+			(at 153.416 105.664 90)
+			(hide yes)
+			(show_name no)
+			(do_not_autoplace no)
+			(effects
+				(font
+					(size 1.27 1.27)
+				)
+			)
+		)
+		(property "Datasheet" ""
+			(at 152.4 105.41 0)
+			(hide yes)
+			(show_name no)
+			(do_not_autoplace no)
+			(effects
+				(font
+					(size 1.27 1.27)
+				)
+			)
+		)
+		(property "Description" "Resistor, US symbol"
+			(at 152.4 105.41 0)
+			(hide yes)
+			(show_name no)
+			(do_not_autoplace no)
+			(effects
+				(font
+					(size 1.27 1.27)
+				)
+			)
+		)
+		(pin "2"
+		)
+		(pin "1"
+		)
+		(instances
+			(project "compactPi"
+				(path "/e63e39d7-6ac0-4ffd-8aa3-1841a4541b55/00000000-0000-0000-0000-00005cff70b1"
+					(reference "R18")
+					(unit 1)
+				)
+			)
+		)
+	)
+	(symbol
 		(lib_id "Connector:HDMI_A_1.4")
 		(at 273.05 105.41 0)
@@
 	(symbol
 		(lib_id "Connector_Generic_MountingPin:Conn_01x04_MountingPin")
-		(at 207.01 153.67 0)
+		(at 218.44 153.67 0)
 		(unit 1)
 		(body_style 1)
@@
 		(dnp no)
 		(property "Reference" "J11"
-			(at 209.55 156.5657 0)
+			(at 220.98 156.5657 0)
 			(show_name no)
 			(do_not_autoplace no)
@@
 		)
 		(property "Value" "Conn_01x04_MountingPin"
-			(at 209.55 154.0257 0)
+			(at 220.98 154.0257 0)
 			(show_name no)
 			(do_not_autoplace no)
@@
 		)
 		(property "Footprint" "Connector_JST:JST_GH_BM04B-GHS-TBT_1x04-1MP_P1.25mm_Vertical"
-			(at 207.01 153.67 0)
+			(at 218.44 153.67 0)
 			(hide yes)
 			(show_name no)
@@
 		)
 		(property "Datasheet" ""
-			(at 207.01 153.67 0)
+			(at 218.44 153.67 0)
 			(hide yes)
 			(show_name no)
@@
 		)
 		(property "Description" "Generic connectable mounting pin connector, single row, 01x04, script generated (kicad-library-utils/schlib/autogen/connector/)"
-			(at 207.01 153.67 0)
+			(at 218.44 153.67 0)
 			(hide yes)
 			(show_name no)
@@
 					(unit 1)
 				)
+			)
+		)
+	)
+	(symbol
+		(lib_id "power:GND")
+		(at 152.4 109.22 0)
+		(unit 1)
+		(body_style 1)
+		(exclude_from_sim no)
+		(in_bom yes)
+		(on_board yes)
+		(in_pos_files yes)
+		(dnp no)
+		(property "Reference" "#PWR0132"
+			(at 152.4 115.57 0)
+			(hide yes)
+			(show_name no)
+			(do_not_autoplace no)
+			(effects
+				(font
+					(size 1.27 1.27)
+				)
+			)
+		)
+		(property "Value" "GND"
+			(at 152.527 113.6142 0)
+			(show_name no)
+			(do_not_autoplace no)
+			(effects
+				(font
+					(size 1.27 1.27)
+				)
+			)
+		)
+		(property "Footprint" ""
+			(at 152.4 109.22 0)
+			(hide yes)
+			(show_name no)
+			(do_not_autoplace no)
+			(effects
+				(font
+					(size 1.27 1.27)
+				)
+			)
+		)
+		(property "Datasheet" ""
+			(at 152.4 109.22 0)
+			(hide yes)
+			(show_name no)
+			(do_not_autoplace no)
+			(effects
+				(font
+					(size 1.27 1.27)
+				)
+			)
+		)
+		(property "Description" "Power symbol creates a global label with name \"GND\" , ground"
+			(at 152.4 109.22 0)
+			(hide yes)
+			(show_name no)
+			(do_not_autoplace no)
+			(effects
+				(font
+					(size 1.27 1.27)
+				)
+			)
+		)
+		(pin "1"
+		)
+		(instances
+			(project "compactPi"
+				(path "/e63e39d7-6ac0-4ffd-8aa3-1841a4541b55/00000000-0000-0000-0000-00005cff70b1"
+					(reference "#PWR0132")
+					(unit 1)
+				)

Commit message: Ehh, mostly there...
Parts:
- C40, C41, R18, R5, R6: KiLib_Generator (none) -> SMD_2terminal_chip_molded
- J11: KiLib_Generator (none) -> connector/SMD_single_row_plus_mounting_pad
- U23: KiLib_Generator (none) -> package/gullwing
Connections:
- net ID_SC is gone; now on net HDMI0_SCL: R6.2
- net ID_SD is gone; now on net HDMI0_SDA: R5.2
- net unconnected-(J11-MountPin-PadMP)_1: now reaches J11.MP (MountPin)
- net GPIO_VREF renamed 3V3
Changed lines of the file:
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@@
 	)
 	(junction
-		(at 280.67 179.07)
-		(diameter 0)
-		(color 0 0 0 0)
-	)
-	(junction
 		(at 63.5 138.43)
 		(diameter 1.016)
@@
 	)
 	(junction
-		(at 273.05 181.61)
-		(diameter 0)
-		(color 0 0 0 0)
-	)
-	(junction
 		(at 129.54 107.95)
 		(diameter 1.016)
@@
 	(wire
 		(pts
-			(xy 251.46 179.07) (xy 280.67 179.07)
-		)
-		(stroke
-			(width 0)
-			(type solid)
-		)
-	)
-	(wire
-		(pts
 			(xy 59.69 95.25) (xy 66.04 95.25)
 		)
@@
 	(wire
 		(pts
-			(xy 251.46 181.61) (xy 273.05 181.61)
-		)
-		(stroke
-			(width 0)
-			(type solid)
-		)
-	)
-	(wire
-		(pts
 			(xy 129.54 123.19) (xy 129.54 115.57)
 		)
@@
 		)
 	)
+	(label "3V3"
+		(at 266.7 163.83 0)
+		(effects
+			(font
+				(size 1.27 1.27)
+			)
+			(justify left bottom)
+		)
+	)
 	(label "HDMI0_D1_N"
 		(at 238.76 92.71 0)
@@
 		)
 	)
-	(label "ID_SC"
-		(at 257.175 179.07 180)
-		(effects
-			(font
-				(size 1.27 1.27)
-			)
-			(justify right bottom)
-		)
-	)
 	(label "HDMI0_D2_P"
 		(at 49.53 171.45 0)
@@
 		)
 	)
-	(label "ID_SD"
-		(at 257.175 181.61 180)
-		(effects
-			(font
-				(size 1.27 1.27)
-			)
-			(justify right bottom)
-		)
-	)
 	(label "USB3-0-TX_N"
 		(at 49.53 133.35 0)
@@
 		)
 	)
-	(label "SCL1"
+	(label "HDMI0_SCL"
 		(at 288.925 179.07 180)
 		(effects
@@
 		)
 	)
-	(label "SDA1"
+	(label "HDMI0_SDA"
 		(at 288.925 181.61 180)
 		(effects
@@
 		)
 	)
-	(label "GPIO_VREF"
-		(at 263.525 163.83 0)
+	(label "HDMI0_SDA"
+		(at 130.81 209.55 0)
 		(effects
 			(font
@@
 		)
 	)
-	(label "HDMI0_SDA"
-		(at 130.81 209.55 0)
+	(label "unconnected-(J11-MountPin-PadMP)_1"
+		(at 218.44 163.83 270)
 		(effects
 			(font
 				(size 1.27 1.27)
 			)
-			(justify left bottom)
+			(justify right bottom)
 		)
 	)
@@
 		)
 	)
-	(hierarchical_label "ID_SC"
-		(shape input)
-		(at 251.46 179.07 180)
-		(effects
-			(font
-				(size 1.27 1.27)
-			)
-			(justify right)
-		)
-	)
 	(hierarchical_label "PCIE_RX_P"
 		(shape input)
@@
 		)
 	)
-	(hierarchical_label "GPIO_VREF"
+	(hierarchical_label "3V3"
 		(shape input)
 		(at 262.89 163.83 180)
@@
 		)
 	)
-	(hierarchical_label "ID_SD"
-		(shape input)
-		(at 251.46 181.61 180)
-		(effects
-			(font
-				(size 1.27 1.27)
-			)
-			(justify right)
-		)
-	)
 	(hierarchical_label "5V0_PERIPHERAL"
 		(shape input)
@@
 			)
 		)
+		(property "KiLib_Generator" "SMD_2terminal_chip_molded"
+			(at 273.05 170.18 0)
+			(hide yes)
+			(show_name no)
+			(do_not_autoplace no)
+			(effects
+				(font
+					(size 1.27 1.27)
+				)
+			)
+		)
 		(pin "1"
 		)
@@
 			)
 		)
+		(property "KiLib_Generator" "SMD_2terminal_chip_molded"
+			(at 280.67 170.18 0)
+			(hide yes)
+			(show_name no)
+			(do_not_autoplace no)
+			(effects
+				(font
+					(size 1.27 1.27)
+				)
+			)
+		)
 		(pin "1"
 		)
@@
 			)
 		)
+		(property "KiLib_Generator" "SMD_2terminal_chip_molded"
+			(at 295.91 210.82 0)
+			(hide yes)
+			(show_name no)
+			(do_not_autoplace no)
+			(effects
+				(font
+					(size 1.27 1.27)
+				)
+			)
+		)
 		(pin "1"
 		)
@@
 			)
 		)
+		(property "KiLib_Generator" "SMD_2terminal_chip_molded"
+			(at 262.89 210.82 0)
+			(hide yes)
+			(show_name no)
+			(do_not_autoplace no)
+			(effects
+				(font
+					(size 1.27 1.27)
+				)
+			)
+		)
 		(pin "1"
 		)
@@
 			)
 		)
+		(property "KiLib_Generator" "SMD_2terminal_chip_molded"
+			(at 152.4 105.41 0)
+			(hide yes)
+			(show_name no)
+			(do_not_autoplace no)
+			(effects
+				(font
+					(size 1.27 1.27)
+				)
+			)
+		)
 		(pin "2"
 		)
@@
 			)
 		)
+		(property "KiLib_Generator" "connector/SMD_single_row_plus_mounting_pad"
+			(at 218.44 153.67 0)
+			(hide yes)
+			(show_name no)
+			(do_not_autoplace no)
+			(effects
+				(font
+					(size 1.27 1.27)
+				)
+			)
+		)
 		(pin "MP"
 		)
@@
 			(at 181.61 154.94 0)
 			(hide yes)
+			(show_name no)
+			(do_not_autoplace no)
+			(effects
+				(font
+					(size 1.27 1.27)
+				)
+			)
+		)
+		(property "KiLib_Generator" "package/gullwing"
+			(at 181.61 154.94 0)
+			(hide yes)
