File: Design Files/Power.kicad_sch (KiCad schematic)
At the start: 66 parts, among them J1 1053101208, U13 TLVM13630RDHR, U14 TLVM13630RDHR, U2 AT24CS64-MAHM, U4 LM74700QDBVRQ1, U5 CSD18511Q5A, U6 CSD18511Q5A, U7 LM74700QDBVRQ1, U8 CSD18511Q5A, U9 LM74700QDBVRQ1

Commit message: New approach
Parts:
- removed C1, C2, C42, C43, C44, C45, C48, C49, C50, C51: 6.8uF, Capacitor_SMD:C_1812_4532Metric, symbol Device:C_Small_US
- removed C4: 47uF, Capacitor_SMD:C_1210_3225Metric, symbol Device:C_Small_US
- added C34: 100nF, Capacitor_SMD:C_0603_1608Metric_Pad1.08x0.95mm_HandSolder, symbol Device:C_Small_US
- U3: footprint TPS25751:TPS25751D -> SiGe_Lib:WQFN38_REF_TEX
Connections:
- net GND: now also C34.2
- net USB_LDO_3V3: now also C34.1
- no-connect marks 8 -> 19
Other:
- moved on the sheet: J1

Commit message: some stuff fixed
Parts:
- added F1, F2: 10A, Fuse:Fuse_1206_3216Metric_Pad1.42x1.75mm_HandSolder, symbol Device:Fuse_Small
- FB1, FB2: footprint (none) -> Inductor_SMD:L_0805_2012Metric
Connections:
- net 5V_PERIPHERAL is gone; now on net 5V0_PERIPHERAL: U3.34 (PP5V), U3.35 (PP5V)
- net V_AUX: now also F2.1; no longer J1.4
- net V_BATT: now also F1.1; no longer J1.1
- new net: F1.2, J1.1
- new net: F2.2, J1.4
Other:
- moved on the sheet: J1
Changed lines of the file:
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@@
 	)
 	(junction
-		(at 231.14 43.18)
+		(at 251.46 43.18)
 		(diameter 0)
 		(color 0 0 0 0)
@@
 	)
 	(no_connect
-		(at 233.68 30.48)
+		(at 254 30.48)
 	)
 	(no_connect
@@
 	)
 	(no_connect
-		(at 233.68 27.94)
+		(at 254 27.94)
 	)
 	(no_connect
@@
 	)
 	(no_connect
-		(at 233.68 38.1)
+		(at 254 38.1)
 	)
 	(no_connect
@@
 	)
 	(no_connect
-		(at 233.68 40.64)
+		(at 254 40.64)
 	)
 	(wire
@@
 	(wire
 		(pts
+			(xy 213.36 33.02) (xy 233.68 33.02)
+		)
+		(stroke
+			(width 0)
+			(type default)
+		)
+	)
+	(wire
+		(pts
 			(xy 151.13 247.65) (xy 154.94 247.65)
 		)
@@
 	(wire
 		(pts
-			(xy 233.68 35.56) (xy 231.14 35.56)
+			(xy 254 35.56) (xy 251.46 35.56)
 		)
 		(stroke
@@
 	(wire
 		(pts
-			(xy 231.14 35.56) (xy 231.14 43.18)
+			(xy 251.46 35.56) (xy 251.46 43.18)
 		)
 		(stroke
@@
 	(wire
 		(pts
-			(xy 213.36 25.4) (xy 233.68 25.4)
-		)
-		(stroke
-			(width 0)
-			(type default)
-		)
-	)
-	(wire
-		(pts
 			(xy 60.96 106.68) (xy 60.96 116.84)
 		)
@@
 	(wire
 		(pts
+			(xy 238.76 25.4) (xy 254 25.4)
+		)
+		(stroke
+			(width 0)
+			(type default)
+		)
+	)
+	(wire
+		(pts
 			(xy 67.31 33.02) (xy 62.23 33.02)
 		)
@@
 	(wire
 		(pts
+			(xy 213.36 25.4) (xy 233.68 25.4)
+		)
+		(stroke
+			(width 0)
+			(type default)
+		)
+	)
+	(wire
+		(pts
 			(xy 92.71 182.88) (xy 92.71 185.42)
 		)
@@
 	(wire
 		(pts
-			(xy 231.14 43.18) (xy 233.68 43.18)
+			(xy 251.46 43.18) (xy 254 43.18)
 		)
 		(stroke
@@
 	(wire
 		(pts
-			(xy 231.14 43.18) (xy 231.14 44.45)
+			(xy 251.46 43.18) (xy 251.46 44.45)
 		)
 		(stroke
@@
 	(wire
 		(pts
-			(xy 64.77 55.88) (xy 64.77 57.15)
+			(xy 238.76 33.02) (xy 254 33.02)
 		)
 		(stroke
@@
 	(wire
 		(pts
-			(xy 66.04 119.38) (xy 60.96 119.38)
+			(xy 64.77 55.88) (xy 64.77 57.15)
 		)
 		(stroke
@@
 	(wire
 		(pts
-			(xy 123.19 116.84) (xy 123.19 118.11)
+			(xy 66.04 119.38) (xy 60.96 119.38)
 		)
 		(stroke
@@
 	(wire
 		(pts
-			(xy 213.36 33.02) (xy 233.68 33.02)
+			(xy 123.19 116.84) (xy 123.19 118.11)
 		)
 		(stroke
@@
 		)
 	)
-	(label "5V_PERIPHERAL"
+	(label "5V0_PERIPHERAL"
 		(at 81.28 217.17 0)
 		(effects
@@
 	)
 	(symbol
+		(lib_id "Device:Fuse_Small")
+		(at 236.22 25.4 0)
+		(unit 1)
+		(body_style 1)
+		(exclude_from_sim no)
+		(in_bom yes)
+		(on_board yes)
+		(in_pos_files yes)
+		(dnp no)
+		(fields_autoplaced yes)
+		(property "Reference" "F1"
+			(at 236.22 20.32 0)
+			(show_name no)
+			(do_not_autoplace no)
+			(effects
+				(font
+					(size 1.27 1.27)
+				)
+			)
+		)
+		(property "Value" "10A"
+			(at 236.22 22.86 0)
+			(show_name no)
+			(do_not_autoplace no)
+			(effects
+				(font
+					(size 1.27 1.27)
+				)
+			)
+		)
+		(property "Footprint" "Fuse:Fuse_1206_3216Metric_Pad1.42x1.75mm_HandSolder"
+			(at 236.22 25.4 0)
+			(hide yes)
+			(show_name no)
+			(do_not_autoplace no)
+			(effects
+				(font
+					(size 1.27 1.27)
+				)
+			)
+		)
+		(property "Datasheet" ""
+			(at 236.22 25.4 0)
+			(hide yes)
+			(show_name no)
+			(do_not_autoplace no)
+			(effects
+				(font
+					(size 1.27 1.27)
+				)
+			)
+		)
+		(property "Description" "Fuse, small symbol"
+			(at 236.22 25.4 0)
+			(hide yes)
+			(show_name no)
+			(do_not_autoplace no)
+			(effects
+				(font
+					(size 1.27 1.27)
+				)
+			)
+		)
+		(pin "1"
+		)
+		(pin "2"
+		)
+		(instances
+			(project "compactPi"
+				(path "/e63e39d7-6ac0-4ffd-8aa3-1841a4541b55/9639513c-40e5-4f7a-bb71-0be3847f4ef3"
+					(reference "F1")
+					(unit 1)
+				)
+			)
+		)
+	)
+	(symbol
 		(lib_id "power:GND")
 		(at 62.23 209.55 0)
@@
 	(symbol
 		(lib_id "power:GND")
-		(at 231.14 44.45 0)
+		(at 251.46 44.45 0)
 		(unit 1)
 		(body_style 1)
@@
 		(fields_autoplaced yes)
 		(property "Reference" "#PWR039"
-			(at 231.14 50.8 0)
+			(at 251.46 50.8 0)
 			(hide yes)
 			(show_name no)
@@
 		)
 		(property "Value" "GND"
-			(at 231.14 49.53 0)
+			(at 251.46 49.53 0)
 			(show_name no)
 			(do_not_autoplace no)
@@
 		)
 		(property "Footprint" ""
-			(at 231.14 44.45 0)
+			(at 251.46 44.45 0)
 			(hide yes)
 			(show_name no)
@@
 		)
 		(property "Datasheet" ""
-			(at 231.14 44.45 0)
+			(at 251.46 44.45 0)
 			(hide yes)
 			(show_name no)
@@
 		)
 		(property "Description" "Power symbol creates a global label with name \"GND\" , ground"
-			(at 231.14 44.45 0)
+			(at 251.46 44.45 0)
 			(hide yes)
 			(show_name no)
@@
 	(symbol
 		(lib_id "SiGe_Lib:1053101208")
-		(at 233.68 25.4 0)
+		(at 254 25.4 0)
 		(unit 1)
 		(body_style 1)
@@
 		(fields_autoplaced yes)
 		(property "Reference" "J1"
-			(at 247.65 33.0199 0)
+			(at 267.97 33.0199 0)
 			(show_name no)
 			(do_not_autoplace no)
@@
 		)
 		(property "Value" "1053101208"
-			(at 247.65 35.5599 0)
+			(at 267.97 35.5599 0)
 			(show_name no)
 			(do_not_autoplace no)
@@
 		)
 		(property "Footprint" "SiGe_Lib:CONN_SD-105310-100_08_MOL"
-			(at 233.68 25.4 0)
+			(at 254 25.4 0)
 			(hide yes)
 			(show_name no)
@@
 		)
 		(property "Datasheet" "https://www.molex.com/en-us/products/part-detail-pdf/1053101208?display=pdf"
-			(at 233.68 25.4 0)
+			(at 254 25.4 0)
 			(hide yes)
 			(show_name no)
@@
 		)
 		(property "Description" ""
-			(at 233.68 25.4 0)
+			(at 254 25.4 0)
 			(hide yes)
 			(show_name no)
@@
 			)
 		)
-		(property "Footprint" ""
+		(property "Footprint" "Inductor_SMD:L_0805_2012Metric"
 			(at 151.13 34.798 90)
 			(hide yes)
@@
 	)
 	(symbol
+		(lib_id "Device:Fuse_Small")
+		(at 236.22 33.02 0)
+		(unit 1)
+		(body_style 1)
+		(exclude_from_sim no)
+		(in_bom yes)
+		(on_board yes)
+		(in_pos_files yes)
+		(dnp no)
+		(fields_autoplaced yes)
+		(property "Reference" "F2"
+			(at 236.22 27.94 0)
+			(show_name no)
+			(do_not_autoplace no)
+			(effects
+				(font
+					(size 1.27 1.27)
+				)
+			)
+		)
+		(property "Value" "10A"
+			(at 236.22 30.48 0)
+			(show_name no)
+			(do_not_autoplace no)
+			(effects
+				(font
+					(size 1.27 1.27)
+				)
+			)
+		)
+		(property "Footprint" "Fuse:Fuse_1206_3216Metric_Pad1.42x1.75mm_HandSolder"
+			(at 236.22 33.02 0)
+			(hide yes)
+			(show_name no)
+			(do_not_autoplace no)
+			(effects
+				(font
+					(size 1.27 1.27)
+				)
+			)
+		)
+		(property "Datasheet" ""
+			(at 236.22 33.02 0)
+			(hide yes)
+			(show_name no)
+			(do_not_autoplace no)
+			(effects
+				(font
+					(size 1.27 1.27)
+				)
+			)
+		)
+		(property "Description" "Fuse, small symbol"
+			(at 236.22 33.02 0)
+			(hide yes)
+			(show_name no)
+			(do_not_autoplace no)
+			(effects
+				(font
+					(size 1.27 1.27)
+				)
+			)
+		)
+		(pin "1"
+		)
+		(pin "2"
+		)
+		(instances
+			(project "compactPi"
+				(path "/e63e39d7-6ac0-4ffd-8aa3-1841a4541b55/9639513c-40e5-4f7a-bb71-0be3847f4ef3"
+					(reference "F2")
+					(unit 1)
+				)
+			)
+		)
+	)
+	(symbol
 		(lib_id "Device:C_Small_US")
 		(at 63.5 137.16 0)
@@
 			)
 		)
-		(property "Footprint" ""
+		(property "Footprint" "Inductor_SMD:L_0805_2012Metric"
 			(at 149.86 118.618 90)
 			(hide yes)

Commit message: major fixes
Parts:
- added C35: 47uF, Capacitor_SMD:C_1210_3225Metric, symbol Device:C_Small_US
- added R15, R16, R17: 10k, Resistor_SMD:R_0402_1005Metric_Pad0.72x0.64mm_HandSolder, symbol Device:R_US
- C25, C27, C6: value 100nF -> 10uF
- R1, R2: value R_US -> 4.7k
- R10, R13: value 53.6k -> 39.2k
Connections:
- net GND: now also C35.2
- net USB_LDO_3V3: now also R15.1, R16.1, R17.1
- net V_USB: now also C35.1
- net at U3.18 (nI2Cc_IRQ): now also R17.2
- net at U3.2 (ADCIN1): now also R15.2
- net at U3.3 (ADCIN2): now also R16.2
- net VIN_3V3 renamed 3V3_IN
- no-connect marks 19 -> 16

Commit message: Ehh, mostly there...
Parts:
- added C37: 22uF, Capacitor_SMD:C_1210_3225Metric, symbol Device:C_Small_US
- added J12: Conn_ARM_SWD_TagConnect_TC2030-NL, Connector:Tag-Connect_TC2030-IDC-NL_2x03_P1.27mm_Vertical, symbol Connector:Conn_ARM_SWD_TagConnect_TC2030-NL
- added R3: 4.7k, Resistor_SMD:R_0402_1005Metric_Pad0.72x0.64mm_HandSolder, symbol Device:R_US
- C10, C11, C12, C13, C14, C15, C16, C17, C18, C19, C20, C21, C22, C23, C24, C26, C28, C29, C30, C31, C32, C33, C34, C46, C47, C5, C6, C7, C8, C9, F1, F2, FB1, FB2, R1, R10, R11, R13, R14, R15, R16, R17, R2, R7, R8, R9: KiLib_Generator (none) -> SMD_2terminal_chip_molded
- C25, C27: KiLib_Generator (none) -> SMD_2terminal_chip_molded; SPN 2679-AGC0603X7R101-104KXPTR-ND -> (none)
- C35: value 47uF -> 22uF; KiLib_Generator (none) -> SMD_2terminal_chip_molded
- U2: value AT24CS64-MAHM -> AT24C256C-SSHL-T; footprint Package_DFN_QFN:DFN-8-1EP_3x2mm_P0.5mm_EP1.3x1.5mm -> SiGe_Lib:8S1_MCH; KiLib_Generator (none) -> package/no_lead
Connections:
- net GND: now also U2.1 (A0), U2.2 (A1), U2.3 (A2), C37.2, J12.5 (GND)
- net I2Cc_SCL: now also J12.4 (SWCLK)
- net I2Cc_SDA: now also J12.2 (SWDIO)
- net LDO_1V5: now also R16.1
- net USB_LDO_3V3: now also J12.1 (VCC), R3.1; no longer R16.1
- net V_USB: now also C37.1
- net EEPROM_WP: now reaches U2.7 (WP)
- net EEPROM_WP: now also J12.6 (SWO), R3.2
- net I2C_PMIC_nINT: now reaches U3.10 (nI2Ct_IRQ)
- net I2C_PMIC_SDA: now reaches U3.8 (I2Ct_SDA)
- net I2C_PMIC_SCL: now reaches U3.9 (I2Ct_SCL)
- no-connect marks 16 -> 14
Other:
- note removed: "ToDos: - [o] Ouput/Input Capacitance - [ ] RT Values for Power Supplies - [ ] Power input protection - [ ] Simulate input protection - [ ] Schematic/Prelim Layout Review"
- moved on the sheet: C24, C25, C27, C34, C35, C5, C6, C7, C8, R1, R15, R16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
