File: Design Files/compactPi.kicad_pcb (KiCad board)
At the start: 6 copper layers, 47 x 105 mm, 153 parts, among them J1 1053101208, J10 Conn_01x06_MountingPin, J11 Conn_01x04_MountingPin, J12 Conn_01x02_MountingPin, J13 Conn_01x02_MountingPin, J14 Micro_SD_Card_Det, J15 USB_C_Receptacle_USB2.0, J16 Conn_01x06_MountingPin, J17 Conn_01x06_MountingPin, J18 Conn_01x06_MountingPin, J19 Conn_01x06_MountingPin, J2 HDMI_A_1.4, J3 Conn_01x04_MountingPin, J4 Conn_01x06_MountingPin, J5 Conn_01x04_MountingPin, J6 Conn_01x04_MountingPin, J7 Conn_01x04_MountingPin, J8 Conn_01x04_MountingPin, J9 Conn_01x04_MountingPin, U1 RT9742GGJ5, U10 BMI270, U11 74LVC2T45DC, U12 74LVC2T45DC, U13 TLVM13630RDHR, U14 TLVM13630RDHR, U15 AK09918C, U16 74LVC2T45DC, U17 RT9742SNGV, U18 PCA9685PW, U2 AT24CS64-MAHM, U20 MMC5983MA, U21 MCP25625x-x-ML, U22 WE-TVS-82400102, U23 WE-TVS-82400102, U24 TCA9517ADGK, U25 BMP390, U4 LM74700QDBVRQ1, U5 CSD18511Q5A, U6 CSD18511Q5A, U7 LM74700QDBVRQ1, U8 CSD18511Q5A, U9 LM74700QDBVRQ1, Y1 Crystal_GND24_Small

Commit message: New approach
Parts:
- removed C1, C2, C42, C43, C44, C45, C48, C49, C50, C51: 6.8uF, Capacitor_SMD:C_1812_4532Metric
- removed C35, C36, C37, C55, C57, C58, C59, C60, C61, C62: 100nF, Capacitor_SMD:C_0402_1005Metric
- removed C4: 47uF, Capacitor_SMD:C_1210_3225Metric
- removed C63: 10uF, Capacitor_SMD:C_0402_1005Metric
- removed G***: LOGO, LOGO
- removed J12, J13: Conn_01x02_MountingPin, Connector_JST:JST_GH_BM02B-GHS-TBT_1x02-1MP_P1.25mm_Vertical
- removed J16, J17, J18, J19: Conn_01x06_MountingPin, Connector_JST:JST_GH_SM06B-GHS-TB_1x06-1MP_P1.25mm_Horizontal
- removed J3: Conn_01x04_MountingPin, Connector_JST:JST_GH_BM04B-GHS-TBT_1x04-1MP_P1.25mm_Vertical
- removed R15, R16, R17, R22: 10k, Resistor_SMD:R_0402_1005Metric_Pad0.72x0.64mm_HandSolder
- removed RN1, RN2, RN3, RN4: R_Pack04, Package_SO:MSOP-8_3x3mm_P0.65mm
- removed U10: BMI270, SiGe_Lib:BMI270_BOS
- removed U11, U12, U16: 74LVC2T45DC, Package_SO:VSSOP-8_2.3x2mm_P0.5mm
- removed U15: AK09918C, SiGe_Lib:BGA4_WL-CSP_AKM
- removed U18: PCA9685PW, Package_SO:TSSOP-28_4.4x9.7mm_P0.65mm
- removed U20: MMC5983MA, SiGe_Lib:MMC5983MA_MEM
- removed U24: TCA9517ADGK, Package_SO:VSSOP-8_3x3mm_P0.65mm
- removed U25: BMP390, SiGe_Lib:10LGA_2X2X0p75_BOS
- C12, C15, C17, C18, C19, C21, C26, C38, C39, C40, C41, C54, C56, C64, C65, C66, C67, D4, J15, NT1, R1, R12, R19, R2, R20, R21, R23, R24, R26, R4, R5, R6, U17, U2, U22, U23: moved to F.Cu
- C34: footprint Capacitor_SMD:C_0402_1005Metric -> Capacitor_SMD:C_0603_1608Metric_Pad1.08x0.95mm_HandSolder; moved to F.Cu
- J14: footprint CM5IO:SDCARD_MOLEX_503398-1892 -> Connector_Card:microSD_HC_Molex_104031-0811
- U3: footprint TPS25751:TPS25751D -> SiGe_Lib:WQFN38_REF_TEX
- moved U1 130.3 mm to (191.2, 155.2), turned to 0 degrees
- moved C3 130.2 mm to (190.9, 158.9), turned to 0 degrees
- moved R26 127.7 mm to (214.7, 153.7)
- moved R24 124.9 mm to (214.7, 149.8)
- moved R23 123.6 mm to (214.7, 147.8)
- moved R12 120.7 mm to (222.8, 103.2), turned to 0 degrees
- moved U23 118.9 mm to (225.8, 120.9)
- moved U22 112.2 mm to (218.8, 104.6), turned to 0 degrees
- moved NT1 108.4 mm to (180.5, 157.7), turned to 0 degrees
- moved C65 105.5 mm to (211.6, 149.4), turned to 0 degrees
- moved C41 105.0 mm to (227.3, 115.7), turned to 0 degrees
- moved C66 101.2 mm to (204.9, 154.7), turned to 0 degrees
- moved R6 101.0 mm to (227.3, 111.8), turned to 0 degrees
- moved R21 100.4 mm to (187.2, 159.7)
- moved C40 100.2 mm to (227.3, 113.8), turned to 0 degrees
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Connections:
- net Net-(U4-GATE) renamed /Power/G_AUX
- net Net-(U4-VCAP) renamed /Power/VCAP_AUX
- net Net-(U5-G) renamed /Power/G_BATT
- net Net-(U7-VCAP) renamed /Power/VCAP_BATT
- net Net-(U8-G) renamed /Power/G_USB
- net Net-(U9-VCAP) renamed /Power/VCAP_USB
- C34 pad 1: /1V8 -> /Power/USB_LDO_3V3
- C41 pad 1: /5V0_PERIPHERAL -> /5V_Peripheral
- J11 pad 1: /5V0_PERIPHERAL -> /5V_Peripheral
- J11 pad 2: /CM5 USB HDMI/USB3-1-D_N -> Net-(J11-Pin_2)
- J11 pad 3: /CM5 USB HDMI/USB3-1-D_P -> Net-(J11-Pin_3)
- U17 pad 1: /5V0_PERIPHERAL -> /5V_Peripheral
- U23 pad 1: unconnected-(U23-Pad1) -> /CM5 USB HDMI/USB3-1-D_N
- U23 pad 3: unconnected-(U23-Pad3) -> /CM5 USB HDMI/USB3-1-D_P
- U23 pad 4: unconnected-(U23-Pad4) -> Net-(J11-Pin_3)
- U23 pad 6: unconnected-(U23-Pad6) -> Net-(J11-Pin_2)
Routing:
- net /CM5 USB HDMI/USB3-1-D_N: track 77.1 -> 0.00 mm, vias 2 -> 0
- net /CM5 USB HDMI/USB3-1-D_P: track 75.9 -> 0.00 mm, vias 2 -> 0
- net /USB2a_P: track 61.8 -> 0.00 mm, vias 1 -> 0
- net /USB2a_N: track 61.7 -> 0.00 mm, vias 1 -> 0
- net /CM5 GPIO Ethernet SDIO/TRD0_N: track 30.2 -> 0.00 mm, vias 1 -> 0
- net /CM5 GPIO Ethernet SDIO/TRD0_P: track 29.4 -> 0.00 mm, vias 1 -> 0
- net /CM5 GPIO Ethernet SDIO/TRD1_P: track 27.5 -> 0.00 mm, vias 1 -> 0
- net /CM5 GPIO Ethernet SDIO/TRD1_N: track 26.7 -> 0.00 mm, vias 1 -> 0
- net /CM5 GPIO Ethernet SDIO/TRD1_RX_N: track 24.4 -> 0.00 mm, vias 1 -> 0
- net /CM5 GPIO Ethernet SDIO/TRD1_RX_P: track 24.3 -> 0.00 mm, vias 1 -> 0
- net /CM5 GPIO Ethernet SDIO/TRD0_TX_N: track 23.2 -> 0.00 mm, vias 1 -> 0
- net /CM5 GPIO Ethernet SDIO/TRD0_TX_P: track 23.1 -> 0.00 mm, vias 1 -> 0
- net /CM5 USB HDMI/HDMI0_D1_N: track 63.5 -> 41.8 mm
- net /CM5 USB HDMI/HDMI0_CK_N: track 59.4 -> 38.4 mm
- net /CM5 USB HDMI/HDMI0_CK_P: track 58.7 -> 39.0 mm
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- added copper zone on B.Cu, net /Power/LDO_1V5
- added copper zone on B.Cu, net /Power/USB_LDO_3V3
- added copper zone on F.Cu, net /Power/USB_LDO_3V3
- added copper zone on B.Cu, net /Power/VIN_3V3
- added copper zone on F.Cu, net /Power/V_AUX
- added copper zone on In2.Cu, net /Power/V_AUX
- added copper zone on F.Cu, net /Power/V_BATT
- added copper zone on In2.Cu, net /Power/V_BATT
- added copper zone on In4.Cu, net /Power/V_COMMON
- added copper zone on In3.Cu, net /Power/V_USB
- added copper zone on In2.Cu, net /VBUS
- removed copper zone on B.Cu, net /1V8
- removed copper zone on B.Cu, net /3V3
- removed copper zone on B.Cu, net /5V0_PERIPHERAL
- removed copper zone on In3.Cu, net /Power/V_COMMON
- removed copper zone on In3.Cu, net /VBUS
- removed copper zone on In1.Cu, net GND
- removed copper zone on In4.Cu, net GND
Other:
- board text removed: "3V3 Sys"
- board text removed: "5V0 Core"
- board text removed: "5V0 Periph"
- board text removed: "ADC"
- board text removed: "CAN"
- board text removed: "Copyright © 2026 Logan Fagg, Licensed under CERN-OHL-S v2"
- board text removed: "ETHER"
- board text removed: "I2C"
- board text removed: "LEAK"
- board text removed: "Pwr In"
- board text removed: "SCL/SDA"
- board text removed: "UART1"
- board text removed: "UART2"
- board text removed: "USB"
- board text removed: "VAUX/G"
- board text removed: "VBATT/G"

Commit message: Checkin
Parts:
- C3, C38, C39, C64, C65, C66, C67, R23, R24, R26, R4, U1, U22: moved to B.Cu
- moved C3 127.9 mm to (106.4, 62.9), turned to 180 degrees
- moved U1 127.6 mm to (106.5, 59.7), turned to 90 degrees
- moved R4 126.1 mm to (106.4, 57.0), turned to 180 degrees
- moved C41 125.9 mm to (122.1, 46.6)
- moved C40 122.4 mm to (122.2, 51.0)
- moved U17 120.3 mm to (123.4, 48.8)
- moved U22 97.8 mm to (130.0, 63.7), turned to 90 degrees
- moved R23 96.8 mm to (118.8, 134.0), turned to 180 degrees
- moved R26 95.5 mm to (122.6, 128.5), turned to 180 degrees
- moved C65 92.5 mm to (120.6, 132.5), turned to 180 degrees
- moved C39 92.0 mm to (119.8, 136.2), turned to -90 degrees
- moved C38 90.4 mm to (121.2, 136.2), turned to -90 degrees
- moved C66 86.7 mm to (120.9, 133.4), turned to 180 degrees
- moved R24 85.7 mm to (131.1, 130.5)
- moved C64 81.8 mm to (131.2, 132.3)
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Connections:
- TR1 pad 1: /CM5 GPIO Ethernet SDIO/TRD1_RX_N -> /CM5 GPIO Ethernet SDIO/TRD1_RX_P
- TR1 pad 14: /CM5 GPIO Ethernet SDIO/TRD1_P -> /CM5 GPIO Ethernet SDIO/TRD1_N
- TR1 pad 16: /CM5 GPIO Ethernet SDIO/TRD1_N -> /CM5 GPIO Ethernet SDIO/TRD1_P
- TR1 pad 3: /CM5 GPIO Ethernet SDIO/TRD1_RX_P -> /CM5 GPIO Ethernet SDIO/TRD1_RX_N
- U22 pad 1: /USB2_N -> /USB2a_N
- U22 pad 3: /USB2_P -> /USB2a_P
- U22 pad 4: /USB2a_P -> /USB2_P
- U22 pad 6: /USB2a_N -> /USB2_N
Routing:
- net /USB2a_N: track 0.00 -> 61.2 mm, vias 0 -> 1
- net /USB2a_P: track 0.00 -> 61.1 mm, vias 0 -> 1
- net /CM5 USB HDMI/HDMI0_HOTPLUG: track 0.00 -> 54.6 mm, vias 0 -> 2
- net /CM5 USB HDMI/HDMI0_CEC: track 0.00 -> 47.2 mm, vias 0 -> 2
- net /CM5 USB HDMI/HDMI0_SCL: track 0.00 -> 38.2 mm, vias 0 -> 2
- net /CM5 USB HDMI/HDMI0_SDA: track 0.00 -> 35.0 mm, vias 0 -> 2
- net /CM5 GPIO Ethernet SDIO/TRD0_TX_P: track 0.00 -> 26.3 mm, vias 0 -> 1
- net /CM5 GPIO Ethernet SDIO/TRD0_TX_N: track 0.00 -> 26.3 mm, vias 0 -> 1
- net /CM5 GPIO Ethernet SDIO/TRD1_RX_N: track 0.00 -> 24.3 mm, vias 0 -> 1
- net /CM5 GPIO Ethernet SDIO/TRD1_RX_P: track 0.00 -> 24.3 mm, vias 0 -> 1
- net /CM5 GPIO Ethernet SDIO/TRD0_P: track 0.00 -> 22.8 mm, vias 0 -> 1
- net /CM5 GPIO Ethernet SDIO/TRD0_N: track 0.00 -> 22.8 mm, vias 0 -> 1
- net /Autopilot Interfaces/CAN_PULL_HI: track 0.00 -> 19.3 mm, vias 0 -> 2
- net /CM5 GPIO Ethernet SDIO/TRD1_N: track 0.00 -> 17.1 mm, vias 0 -> 1
- net /CM5 GPIO Ethernet SDIO/TRD1_P: track 0.00 -> 17.1 mm, vias 0 -> 1
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- added copper zone on In3.Cu, net /5V0_CORE
- added copper zone on B.Cu, net /5V0_PERIPHERAL
- added copper zone on F.Cu, net /5V0_PERIPHERAL
- added copper zone on In3.Cu, net /5V0_PERIPHERAL
- added copper zone on B.Cu, net /Autopilot Interfaces/CAN_PULL_HI
- added copper zone on In1.Cu, net GND
- added copper zone on In3.Cu, net GND
- added copper zone on In4.Cu, net GND

Commit message: some stuff fixed
Parts:
- added F1: 10A, Fuse:Fuse_1206_3216Metric_Pad1.42x1.75mm_HandSolder, F.Cu at (127.3, 56.5)
- added F2: 10A, Fuse:Fuse_1206_3216Metric_Pad1.42x1.75mm_HandSolder, F.Cu at (127.3, 62.3)
- added FB1: FerriteBead_Small, Inductor_SMD:L_0805_2012Metric, B.Cu at (133.5, 91.2)
- added FB2: FerriteBead_Small, Inductor_SMD:L_0805_2012Metric, B.Cu at (118.2, 91.0)
- added R27: 10k, Resistor_SMD:R_0402_1005Metric_Pad0.72x0.64mm_HandSolder, F.Cu at (165.1, 138.2)
- U23: moved to B.Cu
- moved U23 90.7 mm to (135.8, 131.7), turned to -45 degrees
- moved D5 18.3 mm to (122.5, 140.2)
- moved C46 1.60 mm to (124.1, 56.6)
- moved C47 1.60 mm to (124.1, 62.7)
Connections:
- J1 pad 1: /Power/V_BATT -> Net-(F1-Pad2)
- J1 pad 4: /Power/V_AUX -> Net-(F2-Pad2)
- U3 pad 28: /Power/USB_CC1 -> /CC1
- U3 pad 29: /Power/USB_CC2 -> /CC2
- U3 pad 34: /Power/5V_PERIPHERAL -> /5V0_PERIPHERAL
- U3 pad 35: /Power/5V_PERIPHERAL -> /5V0_PERIPHERAL
Routing:
- net /CC2: track 0.00 -> 18.3 mm, vias 0 -> 2
- net /CC1: track 0.00 -> 15.9 mm, vias 0 -> 2
- net /Power/V_COMMON: vias 27 -> 39
- added copper zone on F.Cu, net Net-(F1-Pad2)
- added copper zone on F.Cu, net Net-(F2-Pad2)

Commit message: major fixes
Parts:
- added C69: 10u, Capacitor_SMD:C_0201_0603Metric, F.Cu at (181.7, 164.6)
Connections:
- net Net-(J11-Pin_2) renamed /CM5 USB HDMI/USB3-1-Port_N
- net Net-(J11-Pin_3) renamed /CM5 USB HDMI/USB3-1-Port_P
- C41 pad 1: /5V_Peripheral -> /5V0_PERIPHERAL
- J11 pad 1: /5V_Peripheral -> /5V0_PERIPHERAL
- U17 pad 1: /5V_Peripheral -> /5V0_PERIPHERAL
- U21 pad 3: /5V0_PERIPHERAL -> /3V3
Routing:
- net /5V0_PERIPHERAL: track 1.97 -> 3.25 mm
- net /5V_Peripheral: track 1.28 -> 0.00 mm
Changed lines of the file:
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@@
 		(capping no)
 		(filling no)
+		(zone_defaults)
 		(grid_origin 207.5 79.7)
 		(pcbplotparams
@@
 		)
 	)
+	(footprint "Capacitor_SMD:C_0201_0603Metric"
+		(layer "F.Cu")
+		(at 181.725 164.575)
+		(descr "Capacitor SMD 0201 (0603 Metric), square (rectangular) end terminal, IPC-7351 nominal, (Body size source: https://www.vishay.com/docs/20052/crcw0201e3.pdf)")
+		(tags "capacitor")
+		(property "Reference" "C69"
+			(at 0 -1.05 0)
+			(layer "F.SilkS")
+			(effects
+				(font
+					(size 1 1)
+					(thickness 0.15)
+				)
+			)
+		)
+		(property "Value" "10u"
+			(at 0 1.05 0)
+			(layer "F.Fab")
+			(effects
+				(font
+					(size 1 1)
+					(thickness 0.15)
+				)
+			)
+		)
+		(property "Datasheet" ""
+			(at 0 0 0)
+			(layer "F.Fab")
+			(hide yes)
+			(effects
+				(font
+					(size 1.27 1.27)
+				)
+			)
+		)
+		(property "Description" "capacitor, small US symbol"
+			(at 0 0 0)
+			(layer "F.Fab")
+			(hide yes)
+			(effects
+				(font
+					(size 1.27 1.27)
+				)
+			)
+		)
+		(property "KiLib_Generator" "SMD_2terminal_chip_molded"
+			(at 0 0 0)
+			(layer "F.SilkS")
+			(hide yes)
+			(effects
+				(font
+					(size 1 1)
+					(thickness 0.15)
+				)
+			)
+		)
+		(property ki_fp_filters "C_*")
+		(sheetname "/Autopilot Interfaces/")
+		(sheetfile "autopilot_conn.kicad_sch")
+		(units
+			(unit
+				(name "A")
+				(pins "1" "2")
+			)
+		)
+		(attr smd)
+		(duplicate_pad_numbers_are_jumpers no)
+		(fp_rect
+			(start -0.7 -0.35)
+			(end 0.7 0.35)
+			(stroke
+				(width 0.05)
+				(type solid)
+			)
+			(fill no)
+			(layer "F.CrtYd")
+		)
+		(fp_rect
+			(start -0.3 -0.15)
+			(end 0.3 0.15)
+			(stroke
+				(width 0.1)
+				(type solid)
+			)
+			(fill no)
+			(layer "F.Fab")
+		)
+		(fp_text user "${REFERENCE}"
+			(at 0 -0.68 0)
+			(layer "F.Fab")
+			(effects
+				(font
+					(size 0.25 0.25)
+					(thickness 0.04)
+				)
+			)
+		)
+		(pad "" smd roundrect
+			(at -0.345 0)
+			(size 0.318 0.36)
+			(layers "F.Paste")
+			(roundrect_rratio 0.25)
+		)
+		(pad "" smd roundrect
+			(at 0.345 0)
+			(size 0.318 0.36)
+			(layers "F.Paste")
+			(roundrect_rratio 0.25)
+		)
+		(pad "1" smd roundrect
+			(at -0.32 0)
+			(size 0.46 0.4)
+			(layers "F.Cu" "F.Mask")
+			(roundrect_rratio 0.25)
+			(net "/3V3")
+			(pintype "passive")
+		)
+		(pad "2" smd roundrect
+			(at 0.32 0)
+			(size 0.46 0.4)
+			(layers "F.Cu" "F.Mask")
+			(roundrect_rratio 0.25)
+			(net "GND")
+			(pintype "passive")
+		)
+		(embedded_fonts no)
+		(model "${KICAD10_3DMODEL_DIR}/Capacitor_SMD.3dshapes/C_0201_0603Metric.step"
+			(offset
+				(xyz 0 0 0)
+			)
+			(scale
+				(xyz 1 1 1)
+			)
+			(rotate
+				(xyz 0 0 0)
+			)
+		)
+	)
 	(footprint "Connector_Video:HDMI_Micro-D_Molex_46765-0xxx"
 		(layer "F.Cu")
@@
 			(layers "F.Cu" "F.Mask" "F.Paste")
 			(roundrect_rratio 0.25)
-			(net "/5V_Peripheral")
+			(net "/5V0_PERIPHERAL")
 			(pinfunction "Pin_1_1")
 			(pintype "passive")
@@
 			(layers "F.Cu" "F.Mask" "F.Paste")
 			(roundrect_rratio 0.25)
-			(net "Net-(J11-Pin_2)")
+			(net "/CM5 USB HDMI/USB3-1-Port_N")
 			(pinfunction "Pin_2_2")
 			(pintype "passive")
@@
 			(layers "F.Cu" "F.Mask" "F.Paste")
 			(roundrect_rratio 0.25)
-			(net "Net-(J11-Pin_3)")
+			(net "/CM5 USB HDMI/USB3-1-Port_P")
 			(pinfunction "Pin_3_3")
 			(pintype "passive")
@@
 			(layers "F.Cu" "F.Mask" "F.Paste")
 			(roundrect_rratio 0.25)
-			(net "/5V_Peripheral")
+			(net "/5V0_PERIPHERAL")
 			(pinfunction "IN_1")
 			(pintype "power_in")
@@
 			(layers "F.Cu" "F.Mask" "F.Paste")
 			(roundrect_rratio 0.25)
-			(net "/5V_Peripheral")
+			(net "/5V0_PERIPHERAL")
 			(pintype "passive")
 		)
@@
 			(layers "B.Cu" "B.Mask" "B.Paste")
 			(roundrect_rratio 0.25)
-			(net "Net-(J11-Pin_3)")
+			(net "/CM5 USB HDMI/USB3-1-Port_P")
 			(pintype "passive")
 		)
@@
 			(layers "B.Cu" "B.Mask" "B.Paste")
 			(roundrect_rratio 0.25)
-			(net "Net-(J11-Pin_2)")
+			(net "/CM5 USB HDMI/USB3-1-Port_N")
 			(pintype "passive")
 		)
@@
 			(layers "B.Cu" "B.Mask" "B.Paste")
 			(roundrect_rratio 0.25)
-			(net "/5V0_PERIPHERAL")
+			(net "/3V3")
 			(pinfunction "V_{DD}_3")
 			(pintype "power_in")
@@
 		(width 0.13)
 		(layer "F.Cu")
-		(net "/5V_Peripheral")
+		(net "/5V0_PERIPHERAL")
 	)
 	(segment
@@
 		(width 0.13)
 		(layer "F.Cu")
-		(net "/5V_Peripheral")
+		(net "/5V0_PERIPHERAL")
 	)
 	(via

Commit message: Ehh, mostly there...
Parts:
- removed NT1: NetTie_2, NetTie:NetTie-2_SMD_Pad0.5mm
- added C35: 22uF, Capacitor_SMD:C_1210_3225Metric, F.Cu at (143.2, 62.0)
- added C36: 100nF, Capacitor_SMD:C_0603_1608Metric_Pad1.08x0.95mm_HandSolder, B.Cu at (145.6, 111.2)
- added C37: 22uF, Capacitor_SMD:C_1210_3225Metric, F.Cu at (143.2, 65.2)
- added J12: Conn_ARM_SWD_TagConnect_TC2030-NL, Connector:Tag-Connect_TC2030-IDC-NL_2x03_P1.27mm_Vertical, B.Cu at (141.8, 77.5)
- added R15: 10k, Resistor_SMD:R_0402_1005Metric_Pad0.72x0.64mm_HandSolder, F.Cu at (142.2, 54.2)
- added R16: 10k, Resistor_SMD:R_0402_1005Metric_Pad0.72x0.64mm_HandSolder, F.Cu at (143.7, 54.3)
- added R17: 10k, Resistor_SMD:R_0402_1005Metric_Pad0.72x0.64mm_HandSolder, F.Cu at (141.2, 54.2)
- added R18: 10k, Resistor_SMD:R_0402_1005Metric_Pad0.72x0.64mm_HandSolder, B.Cu at (156.3, 55.5)
- added R22: 4.7k, Resistor_SMD:R_0402_1005Metric_Pad0.72x0.64mm_HandSolder, B.Cu at (155.9, 66.6)
- added R28: 4.7k, Resistor_SMD:R_0402_1005Metric_Pad0.72x0.64mm_HandSolder, B.Cu at (155.9, 64.6)
- added R29: 4.7k, Resistor_SMD:R_0402_1005Metric_Pad0.72x0.64mm_HandSolder, B.Cu at (155.9, 62.6)
- added R3: 4.7k, Resistor_SMD:R_0402_1005Metric_Pad0.72x0.64mm_HandSolder, B.Cu at (137.2, 71.0)
- added R30: 4.7k, Resistor_SMD:R_0402_1005Metric_Pad0.72x0.64mm_HandSolder, B.Cu at (138.6, 107.1)
- added R31: 4.7k, Resistor_SMD:R_0402_1005Metric_Pad0.72x0.64mm_HandSolder, B.Cu at (138.6, 106.1)
- added R32: 4.7k, Resistor_SMD:R_0402_1005Metric_Pad0.72x0.64mm_HandSolder, B.Cu at (138.6, 105.1)
- added U10: AT24C256C-SSHL-T, SiGe_Lib:8S1_MCH, B.Cu at (141.9, 111.3)
- C25, C27, C6: value 100nF -> 10uF
- C34, R5, R6: moved to B.Cu
- R1, R2: value R_US -> 4.7k; moved to B.Cu
- R10, R13: value 53.6k -> 39.2k
- R12: value 2.2K 1% -> 10k
- U2: value AT24CS64-MAHM -> AT24C256C-SSHL-T; footprint Package_DFN_QFN:DFN-8-1EP_3x2mm_P0.5mm_EP1.3x1.5mm -> SiGe_Lib:8S1_MCH; moved to B.Cu
- moved R5 127.6 mm to (109.1, 61.9), turned to -90 degrees
- moved R6 127.2 mm to (110.3, 61.9), turned to -90 degrees
- moved R19 110.4 mm to (139.4, 56.3)
- moved D4 105.0 mm to (139.7, 57.6)
- moved R12 93.4 mm to (140.3, 59.6), turned to 90 degrees
- moved U2 15.6 mm to (133.8, 71.7), turned to 90 degrees
- moved FB2 14.2 mm to (116.2, 105.0), turned to 180 degrees
- moved FB1 14.0 mm to (134.0, 105.2)
- moved C34 11.5 mm to (137.2, 67.7)
- moved R1 10.6 mm to (135.0, 67.0)
- moved C11 10.2 mm to (128.2, 102.5), turned to 180 degrees
- moved R2 9.99 mm to (135.0, 66.0)
- moved C14 9.21 mm to (120.9, 102.5)
- moved R10 5.13 mm to (118.4, 91.8)
- moved R11 5.13 mm to (119.4, 91.8)
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Connections:
- C8 pad 1: /Power/VIN_3V3 -> /3V3
- J10 pad 2: /Autopilot Interfaces/UART2_RX_In -> /Autopilot Interfaces/UART2_TX_Out
- J10 pad 3: /Autopilot Interfaces/UART2_TX_Out -> /Autopilot Interfaces/UART2_RX_In
- J11 pad MP: unconnected-(J11-MountPin-PadMP)_1 -> /CM5 USB HDMI/unconnected-(J11-MountPin-PadMP)_1_1
- J4 pad 2: /Autopilot Interfaces/UART1_RX_In -> /Autopilot Interfaces/UART1_TX_Out
- J4 pad 3: /Autopilot Interfaces/UART1_TX_Out -> /Autopilot Interfaces/UART1_RX_In
- J9 pad MP: unconnected-(J9-MountPin-PadMP)_1 -> /Autopilot Interfaces/unconnected-(J9-MountPin-PadMP)_1_1
- Module1 pad 24: unconnected-(Module1A-GPIO26-Pad24) -> /I2C_PMIC_nINT
- Module1 pad 26: /SPI_CAN_COPI -> /SPI_CAN_CIPO
- Module1 pad 27: /SPI_CAN_CIPO -> /SPI_CAN_COPI
- Module1 pad 30: /I2C_PWM_SDA -> /I2C_PMIC_SDA
- Module1 pad 37: /I2C_PWM_SCL -> /I2C_PMIC_SCL
- Module1 pad 40: /SPI_INT_COPI -> /SPI_INT_CIPO
- Module1 pad 41: /CM5 GPIO Ethernet SDIO/GPIO25 -> /CAN_nINT
- Module1 pad 44: /SPI_INT_CIPO -> /SPI_INT_COPI
- Module1 pad 78: /CM5 GPIO Ethernet SDIO/GPIO_VREF -> /3V3
- Module1 pad 93: GND -> /CM5 GPIO Ethernet SDIO/nRPIBOOT
- R5 pad 1: /CM5 GPIO Ethernet SDIO/GPIO_VREF -> /3V3
- R5 pad 2: /CM5 GPIO Ethernet SDIO/ID_SD -> /CM5 USB HDMI/HDMI0_SDA
- R6 pad 1: /CM5 GPIO Ethernet SDIO/GPIO_VREF -> /3V3
- R6 pad 2: /CM5 GPIO Ethernet SDIO/ID_SC -> /CM5 USB HDMI/HDMI0_SCL
- U2 pad 1: unconnected-(U2-A0-Pad1) -> GND
- U2 pad 2: unconnected-(U2-A1-Pad2) -> GND
- U2 pad 3: unconnected-(U2-A2-Pad3) -> GND
- U2 pad 7: unconnected-(U2-WP-Pad7) -> /Power/EEPROM_WP
- U21 pad 25: /Autopilot Interfaces/SPI_CAN_INT_3V3 -> /CAN_nINT
- U3 pad 10: unconnected-(U3-nI2Ct_IRQ-Pad10) -> /I2C_PMIC_nINT
- U3 pad 18: unconnected-(U3-nI2Cc_IRQ-Pad18) -> Net-(U3-nI2Cc_IRQ)
- U3 pad 2: unconnected-(U3-ADCIN1-Pad2) -> Net-(U3-ADCIN1)
- U3 pad 3: unconnected-(U3-ADCIN2-Pad3) -> Net-(U3-ADCIN2)
- U3 pad 38: /Power/VIN_3V3 -> /3V3
- U3 pad 8: unconnected-(U3-I2Ct_SDA-Pad8) -> /I2C_PMIC_SDA
- U3 pad 9: unconnected-(U3-I2Ct_SCL-Pad9) -> /I2C_PMIC_SCL
Routing:
- net /CM5 GPIO Ethernet SDIO/SD_PWR_ON: track 0.00 -> 76.3 mm, vias 0 -> 2
- net /I2C_EXT_SCL1: track 7.15 -> 68.6 mm, vias 0 -> 2
- net /I2C_EXT_SDA1: track 7.15 -> 67.9 mm, vias 0 -> 2
- net /CAN_nINT: track 0.00 -> 60.2 mm, vias 0 -> 2
- net /SPI_CAN_CE0: track 0.00 -> 57.0 mm, vias 0 -> 2
- net /SPI_CAN_SCK: track 0.00 -> 56.9 mm, vias 0 -> 2
- net /SPI_CAN_COPI: track 0.00 -> 53.2 mm, vias 0 -> 2
- net /SPI_CAN_CIPO: track 0.00 -> 50.2 mm, vias 0 -> 2
- net /Power/I2Cc_SDA: track 3.01 -> 43.7 mm, vias 0 -> 3
- net /Power/I2Cc_SCL: track 1.82 -> 41.4 mm, vias 0 -> 3
- net /CM5 USB HDMI/HDMI0_SDA: track 35.0 -> 53.7 mm, vias 2 -> 3
- net /CM5 USB HDMI/HDMI0_SCL: track 38.2 -> 55.3 mm, vias 2 -> 3
- net /Power/EEPROM_WP: track 0.00 -> 14.3 mm, vias 0 -> 2
- net Net-(U3-nI2Cc_IRQ): track 0.00 -> 13.5 mm, vias 0 -> 2
- net /Power/USB_LDO_3V3: track 0.00 -> 7.40 mm, vias 0 -> 3
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- added copper zone on B.Cu, net /3V3
- added copper zone on In2.Cu, net /3V3
- added copper zone on B.Cu, net /5V0_CORE
- added copper zone on F.Cu, net /5V0_CORE
- added copper zone on In4.Cu, net /5V0_CORE
- added copper zone on In4.Cu, net /Power/USB_LDO_3V3
- added copper zone on F.Cu, net /Power/V_USB
- added copper zone on In1.Cu, net /VBUS
- removed copper zone on F.Cu, net /Power/USB_LDO_3V3
- removed copper zone on B.Cu, net /Power/VIN_3V3
