File: Design Files/compactPi.kicad_pcb (KiCad board)
At the start: 6 copper layers, 47 x 105 mm, 127 parts, among them J1 1053101208, J10 Conn_01x06_MountingPin, J11 Conn_01x04_MountingPin, J12 Conn_ARM_SWD_TagConnect_TC203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, J14 Micro_SD_Card_Det, J15 USB_C_Receptacle_USB2.0, J2 HDMI_A_1.4, J4 Conn_01x06_MountingPin, J5 Conn_01x04_MountingPin, J6 Conn_01x04_MountingPin, J7 Conn_01x04_MountingPin, J8 Conn_01x04_MountingPin, J9 Conn_01x04_MountingPin, U1 RT9742GGJ5, U10 AT24C256C-SSHL-T, U13 TLVM13630RDHR, U14 TLVM13630RDHR, U17 RT9742SNGV, U2 AT24C256C-SSHL-T, U21 MCP25625x-x-ML, U22 WE-TVS-82400102, U23 WE-TVS-82400102, U4 LM74700QDBVRQ1, U5 CSD18511Q5A, U6 CSD18511Q5A, U7 LM74700QDBVRQ1, U8 CSD18511Q5A, U9 LM74700QDBVRQ1, Y1 Crystal_GND24_Small

Commit message: The whole gang is here. And in the board outline
Parts:
- C19, C21, C26, C54, C56, C69, R20, R21, R27: moved to B.Cu
- R22, R28, R29: moved to F.Cu
- moved C19 88.7 mm to (124.8, 74.5)
- moved C26 85.3 mm to (123.2, 90.4)
- moved R21 83.1 mm to (116.4, 116.1), turned to 90 degrees
- moved R20 80.3 mm to (118.4, 116.2), turned to 90 degrees
- moved C21 74.0 mm to (138.6, 83.2), turned to 90 degrees
- moved C56 71.7 mm to (117.5, 118.0), turned to -90 degrees
- moved C69 69.3 mm to (118.6, 136.1), turned to -90 degrees
- moved C54 62.6 mm to (134.5, 110.4)
- moved R27 47.3 mm to (118.4, 130.8), turned to -90 degrees
- moved R22 15.0 mm to (146.9, 54.6), turned to -90 degrees
- moved R28 14.1 mm to (146.0, 54.6), turned to -90 degrees
- moved R29 13.5 mm to (145.0, 54.6), turned to -90 degrees
Routing:
- net Net-(TR1-C_TX): track 0.00 -> 23.4 mm
- net Net-(TR1-C_RD): track 0.00 -> 13.8 mm
- net Net-(TR1-C_RX): track 0.00 -> 7.80 mm
- net /Power/V_COMMON: track 0.00 -> 6.48 mm
- net /I2C_PMIC_SCL: track 1.21 -> 5.81 mm
- net /I2C_PMIC_nINT: track 1.57 -> 5.92 mm
- net /I2C_PMIC_SDA: track 1.19 -> 4.47 mm
- net Net-(C56-Pad1): track 0.00 -> 2.69 mm
- net GND: vias 37 -> 44
